File: kicad/06_dual_active_bridge.kicad_sch (KiCad schematic)
At the start: 0 parts

Commit message: Phase 1: sheets 6 (DAB) and 4 (DC links); diff_amp generalised for TLV316 blocks
Co-Authored-By: Claude Fable 5.1 <noreply@anthropic.com>
Parts:
- added C1, C35, C45, C46, C47, C48, C49, C50: 2.2u, symbol ac_psu:C
- added DAB_PRI_1, DAB_PRI_2, DAB_SEC_1, DAB_SEC_2: PIN, symbol ac_psu:PIN
- added Q10, Q11, Q12, Q9: C3M0065090D, symbol ac_psu:C3M0065090D
- added TR1: ETD34 TRAN 1P1S, symbol ac_psu:ETD34_TRAN_1P1S
Connections:
- new net DAB_CAP_PRI: C1.2, C35.2, C45.1, C46.1, DAB_PRI_2.1, TR1.2 (AB)
- new net DAB_CAP_SEC: C47.2, C48.2, C49.1, C50.1, DAB_SEC_2.1, TR1.4 (SB)
- new net DAB_GATE_HI_PRI: Q9.1 (G)
- new net DAB_GATE_HI_SEC: Q11.1 (G)
- new net DAB_GATE_LO_PRI: Q10.1 (G)
- new net DAB_GATE_LO_SEC: Q12.1 (G)
- new net DAB_GROUND: C49.2, C50.2, Q12.3 (S)
- new net DAB_SOURCE_HI_PRI: DAB_PRI_1.1, Q10.2 (D), Q9.3 (S), TR1.1 (AA)
- new net DAB_SOURCE_HI_SEC: DAB_SEC_1.1, Q11.3 (S), Q12.2 (D), TR1.3 (SA)
- new net DC+: C1.1, C35.1, Q9.2 (D)
- new net ISODC+: C47.1, C48.1, Q11.2 (D)
- new net PGND: C45.2, C46.2, Q10.3 (S)
Other:
- note added: "DC+, PGND, ISODC+ and DAB_GROUND are flagged on sheets 1, 1, 5 and 8."
- note added: "PDF notes: TR1 core 227 nH; winding 52/8/3 || 7/3/3/42."
- note added: "TR1 is not on the PCB (excluded from board): it connects through the DAB_PRI_1/2 and DAB_SEC_1/2 terminals."

Commit message: Phase 2 done: footprints assigned and verified against IPC pads
- tools/gen_footprints.py -> lib/footprint_map.csv + lib/ac_psu.pretty (20 project footprints)
- tools/fpgeom.py: footprint pad loader and rigid fit; tools/check_footprints.py (+ pcbnew
  placement check), added to check_all.sh; reports/footprint_fit.csv for Phase 3 placement
- sch_builder: Footprint field from the map, deterministic UUIDs; all sheets regenerated
- kicad/fp-lib-table; STATUS.md (decisions, residuals, REF3025/C67 findings); Phase 3 prompt

Co-Authored-By: Claude Opus 5.5 <noreply@anthropic.com>
Parts:
- C1, C35, C45, C46, C47, C48, C49, C50: footprint (none) -> Capacitor_SMD:C_2220_5750Metric_Pad1.97x5.40mm_HandSolder
- DAB_PRI_1, DAB_PRI_2, DAB_SEC_1, DAB_SEC_2: footprint (none) -> ac_psu:Terminal_D4.0mm_Drill3.0mm
- Q10, Q11, Q12, Q9: footprint (none) -> Package_TO_SOT_THT:TO-247-3_Vertical
Changed lines of the file:
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@@
 			)
 		)
-		(property "Footprint" ""
+		(property "Footprint" "Capacitor_SMD:C_2220_5750Metric_Pad1.97x5.40mm_HandSolder"
 			(at 28.9052 57.15 0)
 			(effects
@@
 			)
 		)
-		(property "Footprint" ""
+		(property "Footprint" "Capacitor_SMD:C_2220_5750Metric_Pad1.97x5.40mm_HandSolder"
 			(at 39.0652 57.15 0)
 			(effects
@@
 			)
 		)
-		(property "Footprint" ""
+		(property "Footprint" "Capacitor_SMD:C_2220_5750Metric_Pad1.97x5.40mm_HandSolder"
 			(at 28.9052 90.17 0)
 			(effects
@@
 			)
 		)
-		(property "Footprint" ""
+		(property "Footprint" "Capacitor_SMD:C_2220_5750Metric_Pad1.97x5.40mm_HandSolder"
 			(at 39.0652 90.17 0)
 			(effects
@@
 			)
 		)
-		(property "Footprint" ""
+		(property "Footprint" "Package_TO_SOT_THT:TO-247-3_Vertical"
 			(at 81.28 48.26 0)
 			(effects
@@
 			)
 		)
-		(property "Footprint" ""
+		(property "Footprint" "Package_TO_SOT_THT:TO-247-3_Vertical"
 			(at 81.28 86.36 0)
 			(effects
@@
 			)
 		)
-		(property "Footprint" ""
+		(property "Footprint" "ac_psu:Terminal_D4.0mm_Drill3.0mm"
 			(at 27.94 69.85 0)
 			(effects
@@
 			)
 		)
-		(property "Footprint" ""
+		(property "Footprint" "ac_psu:Terminal_D4.0mm_Drill3.0mm"
 			(at 91.44 67.31 0)
 			(effects
@@
 			)
 		)
-		(property "Footprint" ""
+		(property "Footprint" "Package_TO_SOT_THT:TO-247-3_Vertical"
 			(at 137.16 48.26 0)
 			(effects
@@
 			)
 		)
-		(property "Footprint" ""
+		(property "Footprint" "Package_TO_SOT_THT:TO-247-3_Vertical"
 			(at 137.16 86.36 0)
 			(effects
@@
 			)
 		)
-		(property "Footprint" ""
+		(property "Footprint" "Capacitor_SMD:C_2220_5750Metric_Pad1.97x5.40mm_HandSolder"
 			(at 155.9052 57.15 0)
 			(effects
@@
 			)
 		)
-		(property "Footprint" ""
+		(property "Footprint" "Capacitor_SMD:C_2220_5750Metric_Pad1.97x5.40mm_HandSolder"
 			(at 166.0652 57.15 0)
 			(effects
@@
 			)
 		)
-		(property "Footprint" ""
+		(property "Footprint" "Capacitor_SMD:C_2220_5750Metric_Pad1.97x5.40mm_HandSolder"
 			(at 155.9052 90.17 0)
 			(effects
@@
 			)
 		)
-		(property "Footprint" ""
+		(property "Footprint" "Capacitor_SMD:C_2220_5750Metric_Pad1.97x5.40mm_HandSolder"
 			(at 166.0652 90.17 0)
 			(effects
@@
 			)
 		)
-		(property "Footprint" ""
+		(property "Footprint" "ac_psu:Terminal_D4.0mm_Drill3.0mm"
 			(at 154.94 69.85 0)
 			(effects
@@
 			)
 		)
-		(property "Footprint" ""
+		(property "Footprint" "ac_psu:Terminal_D4.0mm_Drill3.0mm"
 			(at 119.38 77.47 0)
 			(effects

Commit message: Phase 3 done: PCB rebuilt from the Proteus gerbers with nets and zones
tools/make_pcb.sh regenerates kicad/ac_psu.kicad_pcb (byte-reproducible):
build_pcb.py (footprints with nets and symbol links at the Proteus
positions, outline, mounting holes, rules), gerber_to_tracks.py (4052
tracks, 173 vias; pour edge strokes recognised and skipped),
assign_nets.py (union-find over copper, 0 shorts/orphans/opens with
pours), pours_to_zones.py (79 zones = Proteus pour copper incl. holes).

New checks in check_all.sh: check_board.py (pads/holes/vias vs IPC),
assign_nets.py --check (after zone fill), drc.py (0 shorts, 0
unconnected, 0 parity issues; courtyard overlaps accepted).

Footprints (user decision): Proteus pad sizes for the headers, TSSOP,
SOT-23(-5), SOIC-16W packages whose KiCad pads shorted/violated
clearance; Proteus pads and drills for TO-247, VXO7805, P27.5 film and
snap-in caps; tighter courtyards for IPC-built footprints.

Co-Authored-By: Claude Opus 5.5 <noreply@anthropic.com>
Parts:
- Q10, Q11, Q12, Q9: footprint Package_TO_SOT_THT:TO-247-3_Vertical -> ac_psu:TO-247-3_Vertical_Proteus
Changed lines of the file:
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@@
 			)
 		)
-		(property "Footprint" "Package_TO_SOT_THT:TO-247-3_Vertical"
+		(property "Footprint" "ac_psu:TO-247-3_Vertical_Proteus"
 			(at 81.28 48.26 0)
 			(effects
@@
 			)
 		)
-		(property "Footprint" "Package_TO_SOT_THT:TO-247-3_Vertical"
+		(property "Footprint" "ac_psu:TO-247-3_Vertical_Proteus"
 			(at 81.28 86.36 0)
 			(effects
@@
 			)
 		)
-		(property "Footprint" "Package_TO_SOT_THT:TO-247-3_Vertical"
+		(property "Footprint" "ac_psu:TO-247-3_Vertical_Proteus"
 			(at 137.16 48.26 0)
 			(effects
@@
 			)
 		)
-		(property "Footprint" "Package_TO_SOT_THT:TO-247-3_Vertical"
+		(property "Footprint" "ac_psu:TO-247-3_Vertical_Proteus"
 			(at 137.16 86.36 0)
 			(effects
