File: kicad/11_signal_isolators.kicad_sch (KiCad schematic)
At the start: 0 parts

Commit message: Phase 1: sheet 11 (signal isolators); builder: rotation-aware fields, text sides, terminals
Co-Authored-By: Claude Fable 5.1 <noreply@anthropic.com>
Parts:
- added C81, C82, C83, C84, C85, C86: 100n, symbol ac_psu:C
- added R22: 39R, symbol ac_psu:R
- added U13, U15, U17: Si8661BD-B-IS, symbol ac_psu:Si8661BD-B-IS
- added U16: Si8660BD-B-IS, symbol ac_psu:Si8660BD-B-IS
Connections:
- new net: R22.1, U15.11 (B5)
- new net 3V3_ISO: C82.2, C83.2, C86.2, U13.1 (VDD1), U15.1 (VDD1), U16.1 (VDD1)
- new net ADASEL0: U15.15 (B1)
- new net ADASEL0_ISO: U15.2 (A1)
- new net ADASEL1: U15.14 (B2)
- new net ADASEL1_ISO: U15.3 (A2)
- new net ADASEL2: U15.13 (B3)
- new net ADASEL2_ISO: U15.4 (A3)
- new net ADCLK: R22.2
- new net ADCLK_ISO: U15.6 (A5)
- new net CLK1: U13.12 (B4)
- new net CLK1_ISO: U13.5 (A4)
- new net CS1: U13.11 (B5)
- new net CS1_ISO: U13.6 (A5)
- new net DAB_PWM_PRI_HI: U16.14 (B2)
- new net DAB_PWM_PRI_HI_ISO: U16.3 (A2)
- new net DAB_PWM_PRI_LO: U16.15 (B1)
- new net DAB_PWM_PRI_LO_ISO: U16.2 (A1)
- new net GND: C81.1, C84.1, C85.1, U13.9 (GND2), U15.9 (GND2), U16.9 (GND2)
- new net GPIO_BYPASS_RLY: U15.12 (B4)
- new net GPIO_BYPASS_RLY_ISOLATED: U15.5 (A4)
- new net ISOGND: C82.1, C83.1, C86.1, U13.8 (GND1), U15.8 (GND1), U16.8 (GND1)
- new net MDATA: U15.10 (B6)
- new net MDATA_ISO: U15.7 (A6)
- new net PWM_G1: U16.12 (B4)
- new net PWM_G1_ISO: U16.5 (A4)
- new net PWM_G2: U16.11 (B5)
- new net PWM_G2_ISO: U16.6 (A5)
- new net PWM_G3: U16.13 (B3)
- new net PWM_G3_ISO: U16.4 (A3)
- new net PWM_G4: U16.10 (B6)
- new net PWM_G4_ISO: U16.7 (A6)
- new net PWM_TRANS1: U13.13 (B3)
- new net PWM_TRANS1_ISO: U13.4 (A3)
- new net PWM_TRANS2: U13.14 (B2)
- new net PWM_TRANS2_ISO: U13.3 (A2)
- new net PWM_TRANS3: U13.15 (B1)
- new net PWM_TRANS3_ISO: U13.2 (A1)
- new net SDATA1: U13.10 (B6)
- new net SDATA1_ISO: U13.7 (A6)
- new net VCC: C81.2, C84.2, C85.2, U13.16 (VDD2), U15.16 (VDD2), U16.16 (VDD2)
- no-connect marks 0 -> 16
Other:
- note added: "3V3 / DC- terminals in the Proteus schematic = nets VCC / GND."
- note added: "U17: spare isolator footprint, not connected (all pins N/C in Proteus)."

Commit message: Phase 2 done: footprints assigned and verified against IPC pads
- tools/gen_footprints.py -> lib/footprint_map.csv + lib/ac_psu.pretty (20 project footprints)
- tools/fpgeom.py: footprint pad loader and rigid fit; tools/check_footprints.py (+ pcbnew
  placement check), added to check_all.sh; reports/footprint_fit.csv for Phase 3 placement
- sch_builder: Footprint field from the map, deterministic UUIDs; all sheets regenerated
- kicad/fp-lib-table; STATUS.md (decisions, residuals, REF3025/C67 findings); Phase 3 prompt

Co-Authored-By: Claude Opus 5.5 <noreply@anthropic.com>
Parts:
- C81, C82, C83, C84, C85, C86: footprint (none) -> Capacitor_SMD:C_0402_1005Metric
- R22: footprint (none) -> Resistor_SMD:R_0402_1005Metric
- U13, U15, U16, U17: footprint (none) -> Package_SO:SOIC-16W_7.5x10.3mm_P1.27mm
Changed lines of the file:
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@@
 			)
 		)
-		(property "Footprint" ""
+		(property "Footprint" "Package_SO:SOIC-16W_7.5x10.3mm_P1.27mm"
 			(at 152.4 50.8 0)
 			(effects
@@
 			)
 		)
-		(property "Footprint" ""
+		(property "Footprint" "Capacitor_SMD:C_0402_1005Metric"
 			(at 93.0148 45.72 0)
 			(effects
@@
 			)
 		)
-		(property "Footprint" ""
+		(property "Footprint" "Capacitor_SMD:C_0402_1005Metric"
 			(at 209.8548 45.72 0)
 			(effects
@@
 			)
 		)
-		(property "Footprint" ""
+		(property "Footprint" "Resistor_SMD:R_0402_1005Metric"
 			(at 106.68 51.562 0)
 			(effects
@@
 			)
 		)
-		(property "Footprint" ""
+		(property "Footprint" "Package_SO:SOIC-16W_7.5x10.3mm_P1.27mm"
 			(at 152.4 96.52 0)
 			(effects
@@
 			)
 		)
-		(property "Footprint" ""
+		(property "Footprint" "Capacitor_SMD:C_0402_1005Metric"
 			(at 108.2548 91.44 0)
 			(effects
@@
 			)
 		)
-		(property "Footprint" ""
+		(property "Footprint" "Capacitor_SMD:C_0402_1005Metric"
 			(at 194.6148 91.44 0)
 			(effects
@@
 			)
 		)
-		(property "Footprint" ""
+		(property "Footprint" "Package_SO:SOIC-16W_7.5x10.3mm_P1.27mm"
 			(at 152.4 142.24 0)
 			(effects
@@
 			)
 		)
-		(property "Footprint" ""
+		(property "Footprint" "Capacitor_SMD:C_0402_1005Metric"
 			(at 108.2548 137.16 0)
 			(effects
@@
 			)
 		)
-		(property "Footprint" ""
+		(property "Footprint" "Capacitor_SMD:C_0402_1005Metric"
 			(at 194.6148 137.16 0)
 			(effects
@@
 			)
 		)
-		(property "Footprint" ""
+		(property "Footprint" "Package_SO:SOIC-16W_7.5x10.3mm_P1.27mm"
 			(at 152.4 187.96 0)
 			(effects

Commit message: Phase 3 done: PCB rebuilt from the Proteus gerbers with nets and zones
tools/make_pcb.sh regenerates kicad/ac_psu.kicad_pcb (byte-reproducible):
build_pcb.py (footprints with nets and symbol links at the Proteus
positions, outline, mounting holes, rules), gerber_to_tracks.py (4052
tracks, 173 vias; pour edge strokes recognised and skipped),
assign_nets.py (union-find over copper, 0 shorts/orphans/opens with
pours), pours_to_zones.py (79 zones = Proteus pour copper incl. holes).

New checks in check_all.sh: check_board.py (pads/holes/vias vs IPC),
assign_nets.py --check (after zone fill), drc.py (0 shorts, 0
unconnected, 0 parity issues; courtyard overlaps accepted).

Footprints (user decision): Proteus pad sizes for the headers, TSSOP,
SOT-23(-5), SOIC-16W packages whose KiCad pads shorted/violated
clearance; Proteus pads and drills for TO-247, VXO7805, P27.5 film and
snap-in caps; tighter courtyards for IPC-built footprints.

Co-Authored-By: Claude Opus 5.5 <noreply@anthropic.com>
Parts:
- U13, U15, U16, U17: footprint Package_SO:SOIC-16W_7.5x10.3mm_P1.27mm -> ac_psu:SOIC-16W_7.5x10.3mm_P1.27mm_Proteus
Changed lines of the file:
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@@
 			)
 		)
-		(property "Footprint" "Package_SO:SOIC-16W_7.5x10.3mm_P1.27mm"
+		(property "Footprint" "ac_psu:SOIC-16W_7.5x10.3mm_P1.27mm_Proteus"
 			(at 152.4 50.8 0)
 			(effects
@@
 			)
 		)
-		(property "Footprint" "Package_SO:SOIC-16W_7.5x10.3mm_P1.27mm"
+		(property "Footprint" "ac_psu:SOIC-16W_7.5x10.3mm_P1.27mm_Proteus"
 			(at 152.4 96.52 0)
 			(effects
@@
 			)
 		)
-		(property "Footprint" "Package_SO:SOIC-16W_7.5x10.3mm_P1.27mm"
+		(property "Footprint" "ac_psu:SOIC-16W_7.5x10.3mm_P1.27mm_Proteus"
 			(at 152.4 142.24 0)
 			(effects
@@
 			)
 		)
-		(property "Footprint" "Package_SO:SOIC-16W_7.5x10.3mm_P1.27mm"
+		(property "Footprint" "ac_psu:SOIC-16W_7.5x10.3mm_P1.27mm_Proteus"
 			(at 152.4 187.96 0)
 			(effects
