File: kicad/10_inu_sdm_relay_drive.kicad_sch (KiCad schematic)
At the start: 0 parts

Commit message: Phase 1: sheet 10 (INU SDM and relay drive)
Co-Authored-By: Claude Fable 5.1 <noreply@anthropic.com>
Parts:
- added C37, C43, C44, C55, C78: 100n, symbol ac_psu:C
- added C51, C54: 220p, symbol ac_psu:C
- added D10, D3, D4, D5: ZLLS400TA, symbol ac_psu:D_Schottky
- added D9: MM3Z5V1T1, symbol ac_psu:D_Zener
- added Q13, Q14: 2N7000, symbol ac_psu:2N7000
- added R50: 33R, symbol ac_psu:R
- added R78, R88, R89, R90: 2.2k, symbol ac_psu:R
- added R92, R93: 10R, symbol ac_psu:R
- added R94: 470R, symbol ac_psu:R
- added U4: ADUM7701-8BRIZ-RL7, symbol ac_psu:ADUM7701-8BRIZ
Connections:
- new net: D10.A, D5.C (K)
- new net: C44.1, Q14.2 (G), R89.1
- new net: D3.C (K), D4.A
- new net: C51.1, R93.1, U4.3 (VIN-)
- new net: C43.1, Q13.2 (G), R78.1
- new net: C55.1, C78.1, D9.C (K), R94.1, U4.1 (VDD1)
- new net: R50.1, U4.6 (MDAT)
- new net: C54.1, R92.1, U4.2 (VIN+)
- new net 20V: D10.C (K)
- new net 20V_ISO_SEC: D4.C (K)
- new net 3V3_ISO: C37.2, U4.8 (VDD2)
- new net GND: C44.2, Q14.3 (S), R90.2
- new net GPIO_BYPASS_RLY: R89.2, R90.1
- new net GPIO_BYPASS_RLY_ISO: R78.2, R88.1
- new net INU_ADCLK: U4.7 (MCLKIN)
- new net INU_SHUNT1: R92.2
- new net INU_SHUNT2: C51.2, C54.2, C55.2, C78.2, D9.A, R93.2, U4.4 (GND1)
- new net ISOGND: C37.1, C43.2, Q13.3 (S), R88.2, U4.5 (GND2)
- new net ISO_AFE_SDM_RAW_VOLTAGE: R94.2
- new net MDATA_INU: R50.2
- new net RELAY_DRIVE: D5.A, Q14.1 (D)
- new net RELAY_DRIVE_ISO: D3.A, Q13.1 (D)
Other:
- note added: "Relay drivers: RELAY_DRIVE -> R20 coil (sheet 1), RELAY_DRIVE_ISO -> R79 coil (sheet 5)."
- note added: "VDD1/GND1 of U4 float on the INU shunt: VDD1 is 5.1 V from D9 via R94 (Proteus auto-named nets), GND1 = INU_SHUNT2."

Commit message: Phase 2 done: footprints assigned and verified against IPC pads
- tools/gen_footprints.py -> lib/footprint_map.csv + lib/ac_psu.pretty (20 project footprints)
- tools/fpgeom.py: footprint pad loader and rigid fit; tools/check_footprints.py (+ pcbnew
  placement check), added to check_all.sh; reports/footprint_fit.csv for Phase 3 placement
- sch_builder: Footprint field from the map, deterministic UUIDs; all sheets regenerated
- kicad/fp-lib-table; STATUS.md (decisions, residuals, REF3025/C67 findings); Phase 3 prompt

Co-Authored-By: Claude Opus 5.5 <noreply@anthropic.com>
Parts:
- C37: footprint (none) -> Capacitor_SMD:C_0402_1005Metric
- C43, C44, C51, C54, C55, C78: footprint (none) -> Capacitor_SMD:C_0603_1608Metric
- D10, D3, D4, D5, D9: footprint (none) -> ac_psu:D_SOD-323_AC
- Q13, Q14: footprint (none) -> ac_psu:SOT-23_Proteus
- R50, R92, R93: footprint (none) -> Resistor_SMD:R_0402_1005Metric
- R78, R88, R89, R90: footprint (none) -> Resistor_SMD:R_0603_1608Metric
- R94: footprint (none) -> Resistor_SMD:R_0805_2012Metric_Pad1.20x1.40mm_HandSolder
- U4: footprint (none) -> ac_psu:SOIC-8W_7.5x5.85mm_P1.27mm_ADuM7701
Changed lines of the file:
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@@
 			)
 		)
-		(property "Footprint" ""
+		(property "Footprint" "ac_psu:SOIC-8W_7.5x5.85mm_P1.27mm_ADuM7701"
 			(at 190.5 50.8 0)
 			(effects
@@
 			)
 		)
-		(property "Footprint" ""
+		(property "Footprint" "Resistor_SMD:R_0402_1005Metric"
 			(at 144.78 46.482 0)
 			(effects
@@
 			)
 		)
-		(property "Footprint" ""
+		(property "Footprint" "Capacitor_SMD:C_0603_1608Metric"
 			(at 153.3652 67.31 0)
 			(effects
@@
 			)
 		)
-		(property "Footprint" ""
+		(property "Footprint" "Resistor_SMD:R_0402_1005Metric"
 			(at 160.02 56.642 0)
 			(effects
@@
 			)
 		)
-		(property "Footprint" ""
+		(property "Footprint" "Capacitor_SMD:C_0603_1608Metric"
 			(at 171.1452 67.31 0)
 			(effects
@@
 			)
 		)
-		(property "Footprint" ""
+		(property "Footprint" "Capacitor_SMD:C_0603_1608Metric"
 			(at 117.8052 58.42 0)
 			(effects
@@
 			)
 		)
-		(property "Footprint" ""
+		(property "Footprint" "Capacitor_SMD:C_0603_1608Metric"
 			(at 107.6452 58.42 0)
 			(effects
@@
 			)
 		)
-		(property "Footprint" ""
+		(property "Footprint" "ac_psu:D_SOD-323_AC"
 			(at 96.52 54.61 0)
 			(effects
@@
 			)
 		)
-		(property "Footprint" ""
+		(property "Footprint" "Resistor_SMD:R_0805_2012Metric_Pad1.20x1.40mm_HandSolder"
 			(at 83.82 36.322 0)
 			(effects
@@
 			)
 		)
-		(property "Footprint" ""
+		(property "Footprint" "Resistor_SMD:R_0402_1005Metric"
 			(at 218.44 52.578 0)
 			(effects
@@
 			)
 		)
-		(property "Footprint" ""
+		(property "Footprint" "Capacitor_SMD:C_0402_1005Metric"
 			(at 253.0348 46.99 0)
 			(effects
@@
 			)
 		)
-		(property "Footprint" ""
+		(property "Footprint" "ac_psu:SOT-23_Proteus"
 			(at 93.98 129.54 0)
 			(effects
@@
 			)
 		)
-		(property "Footprint" ""
+		(property "Footprint" "ac_psu:D_SOD-323_AC"
 			(at 83.82 124.46 0)
 			(effects
@@
 			)
 		)
-		(property "Footprint" ""
+		(property "Footprint" "ac_psu:D_SOD-323_AC"
 			(at 71.12 124.46 0)
 			(effects
@@
 			)
 		)
-		(property "Footprint" ""
+		(property "Footprint" "Capacitor_SMD:C_0603_1608Metric"
 			(at 82.2452 142.24 0)
 			(effects
@@
 			)
 		)
-		(property "Footprint" ""
+		(property "Footprint" "Resistor_SMD:R_0603_1608Metric"
 			(at 73.66 130.302 0)
 			(effects
@@
 			)
 		)
-		(property "Footprint" ""
+		(property "Footprint" "Resistor_SMD:R_0603_1608Metric"
 			(at 61.722 138.43 0)
 			(effects
@@
 			)
 		)
-		(property "Footprint" ""
+		(property "Footprint" "ac_psu:SOT-23_Proteus"
 			(at 246.38 129.54 0)
 			(effects
@@
 			)
 		)
-		(property "Footprint" ""
+		(property "Footprint" "ac_psu:D_SOD-323_AC"
 			(at 236.22 124.46 0)
 			(effects
@@
 			)
 		)
-		(property "Footprint" ""
+		(property "Footprint" "ac_psu:D_SOD-323_AC"
 			(at 223.52 124.46 0)
 			(effects
@@
 			)
 		)
-		(property "Footprint" ""
+		(property "Footprint" "Capacitor_SMD:C_0603_1608Metric"
 			(at 234.6452 142.24 0)
 			(effects
@@
 			)
 		)
-		(property "Footprint" ""
+		(property "Footprint" "Resistor_SMD:R_0603_1608Metric"
 			(at 226.06 130.302 0)
 			(effects
@@
 			)
 		)
-		(property "Footprint" ""
+		(property "Footprint" "Resistor_SMD:R_0603_1608Metric"
 			(at 214.122 138.43 0)
 			(effects

Commit message: v4 design fixes: RET_ISO->ISOGND, U11 INH->GND, C88/C89 on ADA2/ADA3, ADuM7701 RC compensation, R48 Kelvin split
Board frozen: kicad/ac_psu.kicad_pcb edited by one-shot pcbnew scripts tools/v4/fix_1..5
(apply_all.sh, reproducible from the tag's board); make_pcb.sh rebuilds the Proteus board from
tag proteus-conversion-complete into build/proteus/ (byte-identical, checked by regen_check).
Proteus comparisons apply exactly lib/v4_deviations.csv + lib/v4_copper.csv (tools/deviations.py,
wrappers compare_netlists_v4 / check_symbols_v4, deviation support in check_board,
check_footprints, gen_footprints, ipc356_diff, gerber_roundtrip). p2k submodule unchanged.
check_all: ALL CHECKS PASSED; DRC 0 shorts / 0 unconnected / 0 parity (+1 accepted courtyard
overlap C91/U5).

Co-Authored-By: Claude Opus 5.5 <noreply@anthropic.com>
Parts:
- added C90: 100n C0G, Capacitor_SMD:C_1206_3216Metric, symbol ac_psu:C
- R92, R93: value 10R -> 12.4R
Connections:
- net at C54.1, R92.1, U4.2 (VIN+): now also C90.1
- net at C51.1, R93.1, U4.3 (VIN-): now also C90.2
Other:
- note added: "tau = L/R = 2.5 us; with 100 nF use R_leg = 2.5 Ohm per nH of shunt L (4 nH -> 10R, 5 nH -> 12.4R, 6 nH -> 15R)."
- note added: "v4: C90 100n C0G (1206) across VIN+/VIN- compensates the shunt inductance:"
Changed lines of the file:
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@@
 			)
 		)
-		(property "Value" "10R"
+		(property "Value" "12.4R"
 			(at 144.78 46.23 90)
 			(effects
@@
 			)
 		)
-		(property "Value" "10R"
+		(property "Value" "12.4R"
 			(at 160.02 62.23 90)
 			(effects
@@
 	)
 	(symbol
+		(lib_id "ac_psu:C")
+		(at 166.37 53.34 0)
+		(unit 1)
+		(exclude_from_sim no)
+		(in_bom yes)
+		(on_board yes)
+		(dnp no)
+		(property "Reference" "C90"
+			(at 170.56 52.07 0)
+			(effects
+				(font
+					(size 1.27 1.27)
+				)
+			)
+		)
+		(property "Value" "100n C0G"
+			(at 173.31 54.61 0)
+			(effects
+				(font
+					(size 1.27 1.27)
+				)
+			)
+		)
+		(property "Footprint" "Capacitor_SMD:C_1206_3216Metric"
+			(at 167.3352 57.15 0)
+			(effects
+				(font
+					(size 1.27 1.27)
+				)
+				(hide yes)
+			)
+		)
+		(property "Datasheet" ""
+			(at 166.37 53.34 0)
+			(effects
+				(font
+					(size 1.27 1.27)
+				)
+				(hide yes)
+			)
+		)
+		(property "Description" "Unpolarized capacitor"
+			(at 166.37 53.34 0)
+			(effects
+				(font
+					(size 1.27 1.27)
+				)
+				(hide yes)
+			)
+		)
+		(pin "1"
+		)
+		(pin "2"
+		)
+		(instances
+			(project "ac_psu"
+				(path "/04fb09b4-531d-41de-805c-3ed4ed6dcfa8/2d66ecaa-c50e-45f5-a456-6f9e5dc4a618"
+					(reference "C90")
+					(unit 1)
+				)
+			)
+		)
+	)
+	(wire
+		(pts
+			(xy 166.37 48.26) (xy 166.37 49.53)
+		)
+		(stroke
+			(width 0)
+			(type default)
+		)
+	)
+	(junction
+		(at 166.37 48.26)
+		(diameter 0)
+		(color 0 0 0 0)
+	)
+	(wire
+		(pts
+			(xy 166.37 57.15) (xy 166.37 58.42)
+		)
+		(stroke
+			(width 0)
+			(type default)
+		)
+	)
+	(junction
+		(at 166.37 58.42)
+		(diameter 0)
+		(color 0 0 0 0)
+	)
+	(text "v4: C90 100n C0G (1206) across VIN+/VIN- compensates the shunt inductance:"
+		(exclude_from_sim no)
+		(at 71.12 85.09 0)
+		(effects
+			(font
+				(size 1.27 1.27)
+			)
+			(justify left bottom)
+		)
+	)
+	(text "tau = L/R = 2.5 us; with 100 nF use R_leg = 2.5 Ohm per nH of shunt L (4 nH -> 10R, 5 nH -> 12.4R, 6 nH -> 15R)."
+		(exclude_from_sim no)
+		(at 71.12 88.9 0)
+		(effects
+			(font
+				(size 1.27 1.27)
+			)
+			(justify left bottom)
+		)
+	)
+	(symbol
