File: kicad/ac_psu.kicad_pcb (KiCad board)
At the start: 4 copper layers, 246.8 x 154.7 mm, 271 parts, among them J1 HB GT CONNECTOR, J10 PIN, J11 38 PIN HEADER 50TH, J12 2X3 PIN 50TH CONNECTOR, J2 HB GT CONNECTOR, J3 HB GT CONNECTOR, J4 HB GT CONNECTOR, J5 PIN, J6 HB GT CONNECTOR, J7 PIN, J8 HB GT CONNECTOR, J9 PIN, Q1 C3M0065090D, Q10 C3M0065090D, Q11 C3M0065090D, Q12 C3M0065090D, Q13 2N7000, Q14 2N7000, Q2 C3M0065090D, Q3 C3M0065090D, Q4 C3M0065090D, Q5 C3M0065090D, Q6 C3M0065090D, Q7 C3M0065090D, Q8 C3M0065090D, Q9 C3M0065090D, U1 OPA2353UA, U10 TPS73033DBVT, U11 SN74LV4051, U12 TLV316IDBVR, U13 Si8661BD-B-IS, U14 TLV316IDBVR, U15 Si8661BD-B-IS, U16 Si8660BD-B-IS, U17 Si8661BD-B-IS, U2 TLV316IDBVR, U3 TPS73033DBVT, U4 ADUM7701-8BRIZ-RL7, U5 ADUM7701-8BRIZ-RL7, U6 ADUM7701-8BRIZ-RL7, U7 OPA2353UA, U8 VXO7805-1000, U9 VXO7805-500

Commit message: v4 design fixes: RET_ISO->ISOGND, U11 INH->GND, C88/C89 on ADA2/ADA3, ADuM7701 RC compensation, R48 Kelvin split
Board frozen: kicad/ac_psu.kicad_pcb edited by one-shot pcbnew scripts tools/v4/fix_1..5
(apply_all.sh, reproducible from the tag's board); make_pcb.sh rebuilds the Proteus board from
tag proteus-conversion-complete into build/proteus/ (byte-identical, checked by regen_check).
Proteus comparisons apply exactly lib/v4_deviations.csv + lib/v4_copper.csv (tools/deviations.py,
wrappers compare_netlists_v4 / check_symbols_v4, deviation support in check_board,
check_footprints, gen_footprints, ipc356_diff, gerber_roundtrip). p2k submodule unchanged.
check_all: ALL CHECKS PASSED; DRC 0 shorts / 0 unconnected / 0 parity (+1 accepted courtyard
overlap C91/U5).

Co-Authored-By: Claude Opus 5.5 <noreply@anthropic.com>
Parts:
- added C88: 1n, Capacitor_SMD:C_0402_1005Metric, B.Cu at (60.1, 9.35)
- added C89: 1n, Capacitor_SMD:C_0402_1005Metric, B.Cu at (57.6, 8.03)
- added C90: 100n C0G, Capacitor_SMD:C_1206_3216Metric, B.Cu at (10.2, -37.3)
- added C91: 100n C0G, Capacitor_SMD:C_1206_3216Metric, B.Cu at (8.10, 64.0)
- added C92: 100n C0G, Capacitor_SMD:C_1206_3216Metric, B.Cu at (108.6, -33.0)
- R57, R58, R73, R74, R92, R93: value 10R -> 12.4R
Connections:
- C15 pad 2: RET_ISO -> ISOGND
- C36 pad 2: RET_ISO -> ISOGND
- J5 pad 1: SHUNT1 -> /01 afe/SHUNT1_FORCE
- R48 pad 3: SHUNT1 -> /01 afe/SHUNT1_FORCE
- R49 pad 1: RET_ISO -> ISOGND
- TR2 pad 6: RET_ISO -> ISOGND
- U11 pad 6: DGND -> GND
Routing:
- net SHUNT1: track 35.3 -> 23.0 mm
- net Net-(U5-VIN-): track 5.69 -> 12.7 mm, vias 0 -> 2
- net Net-(U4-VIN-): track 5.29 -> 12.2 mm, vias 0 -> 2
- net /01 afe/SHUNT1_FORCE: track 0.00 -> 6.12 mm
- net RET_ISO: track 5.59 -> 0.00 mm, vias 2 -> 0
- net ISOGND: track 288.6 -> 294.2 mm, vias 17 -> 22
- net Net-(U4-VIN+): track 7.57 -> 11.4 mm
- net Net-(U6-VIN+): track 7.57 -> 10.1 mm, vias 0 -> 1
- net GND: track 456.4 -> 458.7 mm, vias 25 -> 27
- net Net-(U6-VIN-): track 5.35 -> 7.32 mm, vias 0 -> 1
- net Net-(U5-VIN+): track 7.74 -> 9.46 mm
- net ADA2: track 11.9 -> 12.7 mm, vias 0 -> 1
- net ADA3: track 16.2 -> 17.0 mm, vias 0 -> 1
- added copper zone on B.Cu, net /01 afe/SHUNT1_FORCE
- added copper zone on B.Cu, net ISOGND
- removed copper zone on B.Cu, net RET_ISO
- removed copper zone on F.Cu, net RET_ISO
- removed copper zone on B.Cu, net SHUNT1
