File: kicad/ac_psu.kicad_pcb (KiCad board)
At the start: 4 copper layers, 246.8 x 154.7 mm, 276 parts, among them J1 HB GT CONNECTOR, J10 PIN, J11 38 PIN HEADER 50TH, J12 2X3 PIN 50TH CONNECTOR, J2 HB GT CONNECTOR, J3 HB GT CONNECTOR, J4 HB GT CONNECTOR, J5 PIN, J6 HB GT CONNECTOR, J7 PIN, J8 HB GT CONNECTOR, J9 PIN, Q1 C3M0065090D, Q10 C3M0065090D, Q11 C3M0065090D, Q12 C3M0065090D, Q13 2N7000, Q14 2N7000, Q2 C3M0065090D, Q3 C3M0065090D, Q4 C3M0065090D, Q5 C3M0065090D, Q6 C3M0065090D, Q7 C3M0065090D, Q8 C3M0065090D, Q9 C3M0065090D, U1 OPA2353UA, U10 TPS73033DBVT, U11 SN74LV4051, U12 TLV316IDBVR, U13 Si8661BD-B-IS, U14 TLV316IDBVR, U15 Si8661BD-B-IS, U16 Si8660BD-B-IS, U17 Si8661BD-B-IS, U2 TLV316IDBVR, U3 TPS73033DBVT, U4 ADUM7701-8BRIZ-RL7, U5 ADUM7701-8BRIZ-RL7, U6 ADUM7701-8BRIZ-RL7, U7 OPA2353UA, U8 VXO7805-1000, U9 VXO7805-500

Commit message: v4: R19/R32 422R instead of 420R (not E96, not stocked at JLC), fix 9
2.5 V x 820/(422+820) = 1.6506 V (420R: 1.6532 V). Deviation value rows,
sheet 3 note, board values.

Co-Authored-By: Claude Opus 5.5 <noreply@anthropic.com>
Claude-Session: https://claude.ai/code/session_01Am5hpeWpvZbzmHWspFiWJm
Parts:
- R19, R32: value 420R -> 422R
Changed lines of the file:
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@@
 			)
 		)
-		(property "Value" "420R"
+		(property "Value" "422R"
 			(at 0 1.17 90)
 			(layer "F.Fab")
@@
 			)
 		)
-		(property "Value" "420R"
+		(property "Value" "422R"
 			(at 0 1.17 0)
 			(layer "F.Fab")

Commit message: v4 fix 10: U8 K7805-2000R3 (5 V / 2 A) with C93/C94 per its datasheet
For the isolated control card (efinix_soc_board POWER_BUDGET.md): U8 value
VXO7805-1000 -> Mornsun K7805-2000R3 (same SIP-3 pinout and footprint, U9
unchanged). C93 10u 50V X7R 1210 (22u 50V not stocked in 1206/1210) at pin 1,
C94 22u 10V 0805 at pin 3, bottom side just south of U8's pins with short
B.Cu tracks; pin 2 is on the In1 ISOGND zone. Deviation rows (value, 2 parts,
4 pins, B.Cu area), sheet 3, part map. Footprint courtyard 0.075 mm short of
the K7805's 6.85 mm body depth (kept, noted).

Co-Authored-By: Claude Opus 5.5 <noreply@anthropic.com>
Claude-Session: https://claude.ai/code/session_01Am5hpeWpvZbzmHWspFiWJm
Parts:
- added C93: 10u 50V, Capacitor_SMD:C_1210_3225Metric, B.Cu at (105.4, 22.9)
- added C94: 22u 10V, Capacitor_SMD:C_0805_2012Metric, B.Cu at (109.4, 23.3)
- U8: value VXO7805-1000 -> K7805-2000R3
Routing:
- net ISOGND: track 294.2 -> 300.7 mm
- net 20V_ISO_SEC: track 385.0 -> 388.2 mm
- net 5V_ISOL: track 198.8 -> 201.1 mm

Commit message: v4 fix 11/12: measurement filters (reports/noise findings 1-5), AMC1306M05
Schematic (sheets 1/3/4/5/9): C95-C106 1n C0G across every 10k leg of the six
difference amplifiers (15.9 kHz tap-node filter), R7 1k -> 10k (U1B + leg
matched; ADA3 scaling changes), R18/R9 100R -> 8.2k with C88/C89 4.7n C0G and
new C107/C108 4.7n on ISOADA1/2 (4.1 kHz), C42/C2 1n -> 10n C0G (1.9 kHz DC
links), C109/C110 100n on REF_1V65/REF_1V65_ISO. R64/DAB series R unchanged
(L unknown; 25R per leg for 10 nH).
Board: fix 11 places the 16 caps (10 top beside their resistor, 6 bottom with
7 vias), renames six auto-named output nets, sets the values; fix 12 re-runs
fix 8's silk placement. DRC 293 (+1 silk), 0 shorts/unconnected/parity.
Deviation rows, v4_copper vias/areas, part map. Replay of fixes 1-12 on the
tag's board gives the board and edit log.
fab: C0G codes C307441/C1518204/C22400107, U4-U6 AMC1306M05DWVR (C701717,
+-50 mV, 4.9k R_IND, checked in SBAS734D), CPL 205 parts, stock for 5 boards
(AMC1306M05: 5 in stock). Noise report: CMTI 50 kV/us min correction.

Co-Authored-By: Claude Opus 5.5 <noreply@anthropic.com>
Claude-Session: https://claude.ai/code/session_01Am5hpeWpvZbzmHWspFiWJm
Parts:
- added C100: 1n C0G, Capacitor_SMD:C_0402_1005Metric, B.Cu at (59.3, 15.3)
- added C101: 1n C0G, Capacitor_SMD:C_0402_1005Metric, F.Cu at (88.8, -38.1)
- added C102: 1n C0G, Capacitor_SMD:C_0402_1005Metric, F.Cu at (95.0, -35.9)
- added C103: 1n C0G, Capacitor_SMD:C_0402_1005Metric, F.Cu at (74.5, -36.9)
- added C104: 1n C0G, Capacitor_SMD:C_0402_1005Metric, F.Cu at (74.5, -38.8)
- added C105: 1n C0G, Capacitor_SMD:C_0402_1005Metric, F.Cu at (79.1, -35.2)
- added C106: 1n C0G, Capacitor_SMD:C_0402_1005Metric, B.Cu at (82.9, -37.5)
- added C107: 4.7n C0G, Capacitor_SMD:C_0402_1005Metric, B.Cu at (77.8, -41.0)
- added C108: 4.7n C0G, Capacitor_SMD:C_0402_1005Metric, F.Cu at (84.8, -40.2)
- added C109: 100n, Capacitor_SMD:C_0402_1005Metric, F.Cu at (53.9, -4.40)
- added C110: 100n, Capacitor_SMD:C_0402_1005Metric, F.Cu at (114.0, -12.4)
- added C95: 1n C0G, Capacitor_SMD:C_0402_1005Metric, F.Cu at (53.8, 6.44)
- added C96: 1n C0G, Capacitor_SMD:C_0402_1005Metric, B.Cu at (50.7, 6.90)
- added C97: 1n C0G, Capacitor_SMD:C_0402_1005Metric, F.Cu at (53.8, 0.14)
- added C98: 1n C0G, Capacitor_SMD:C_0402_1005Metric, B.Cu at (51.2, -1.10)
- added C99: 1n C0G, Capacitor_SMD:C_0402_1005Metric, B.Cu at (62.0, 14.3)
- C2, C42: value 1n -> 10n C0G
- C88, C89: value 1n -> 4.7n C0G
- R18, R9: value 100 -> 8.2k
- R7: value 1k -> 10k
Routing:
- net ISOGND: track 300.7 -> 304.2 mm, vias 22 -> 23
- net REF_1V65_ISO: track 59.8 -> 62.9 mm
- net REF_1V65: track 11.2 -> 14.2 mm
- net GND: track 458.7 -> 460.9 mm
- net ISOADA2: track 51.0 -> 52.6 mm
- net Net-(U14-+): track 6.04 -> 7.20 mm
- net Net-(C98-Pad1): track 2.80 -> 3.90 mm, vias 0 -> 1
- net Net-(U1B-+): track 9.75 -> 10.8 mm
- net Net-(U7B-+): track 105.0 -> 106.0 mm
- net Net-(U1A-+): track 84.6 -> 85.6 mm
- net Net-(U2-+): track 130.4 -> 131.4 mm
- net Net-(U7A--): track 90.5 -> 91.5 mm
- net Net-(U7A-+): track 90.8 -> 91.8 mm
- net Net-(C104-Pad1): track 2.98 -> 3.98 mm
- net Net-(C102-Pad1): track 3.60 -> 4.60 mm
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