File: kicad/07_auxiliary_supply.kicad_sch (KiCad schematic)
At the start: 0 parts

Commit message: Phase 1 done: sheet 7 (aux supply), strict check_all, STATUS and Phase 2 handoff prompt
Co-Authored-By: Claude Fable 5.1 <noreply@anthropic.com>
Parts:
- added C15, C28: 220u, symbol ac_psu:C_Polarized
- added C36, C41, C65, C66: 4.7u, symbol ac_psu:C
- added C57, C58: 22u, symbol ac_psu:C
- added C62: 470p, symbol ac_psu:C
- added C63: 22pF, symbol ac_psu:C
- added C67: 100u, symbol ac_psu:C_Polarized
- added C68: 100n, symbol ac_psu:C
- added D1, D2: ES1A, symbol ac_psu:D
- added D6: S1M, symbol ac_psu:D
- added D7: ZLLS400TA, symbol ac_psu:D_Schottky
- added PWM1: IW1830, symbol ac_psu:IW1830
- added R23: 100R, symbol ac_psu:R
- added R24, R33, R34, R43: 1M, symbol ac_psu:R
- added R25: 15k, symbol ac_psu:R
- added R26: NA, symbol ac_psu:R
- added R29: 1.2k, symbol ac_psu:R
- added R31: 1k, symbol ac_psu:R
- added R44: 39k, symbol ac_psu:R
- added R45, R47: 2.49R, symbol ac_psu:R
- added R49: 12.1K, symbol ac_psu:R
- added TR2: EF20_AUX_TRANS, symbol ac_psu:EF20_AUX_TRANS
Connections:
- new net: C62.2, R23.1, R24.2
- new net: D6.C (K), R23.2
- new net: C65.1, C66.1, D7.C (K), PWM1.1 (Vcc), R33.2
- new net: R34.1, R43.2
- new net: D1.A, TR2.7
- new net: PWM1.2 (Vsense), R31.1
- new net: R33.1, R34.2
- new net 20V: C28.1, C41.1, D2.C (K), D7.A
- new net 20V_ISO_SEC: C15.1, C36.1, D1.C (K), R49.2
- new net 5V: C57.2, C58.2, C67.2
- new net AUX_FB: D2.A, R25.1, R44.1, TR2.3
- new net AUX_FEEDBACK: C63.2, R25.2, R26.1, R29.1, R31.2, R44.2
- new net AUX_ISENSE: PWM1.4 (I_sense), PWM1.5 (S), R45.1, R47.1
- new net AUX_SWITCH_NODE: D6.A, PWM1.7 (D), PWM1.8 (D), TR2.2
- new net DC+: C62.1, C68.2, R24.1, R43.1, TR2.1
- new net GND: C28.2, C41.2, C57.1, C58.1, C63.1, C65.2, C66.2, C67.1, C68.1, PWM1.3 (GND), R26.2, R29.2, R45.2, R47.2, TR2.4
- new net RET_ISO: C15.2, C36.2, R49.1, TR2.6
- no-connect marks 0 -> 4
Other:
- note added: "C67: IPC pin 1 is on GND (C28/C15 have pin 1 on the + rail) - check footprint polarity in Phase 2."
- note added: "PDF notes: vsense nominal = 1.536 V, vsense OVP threshold = 1.838 V, Isense pk = 1 V, Vpeak = 520 V"
- note added: "R26: NA (not fitted) in the PDF."
- note added: "TR1 : core 227 nH, 52/8/3 || 7/3/3/42 (note printed on this page, TR1 is on sheet 6)"
- note added: "The PDF's ISO_GND terminal is wired to RET_iso: net RET_ISO (not ISOGND). 20V_ISO_SEC feeds U8 (sheet 3) and the"
- note added: "Vsense @ 1.536 V = 5.8368 Vaux; Isense ocp = 1.15 V; V5.1; 'R64 = 39k / v2 trans' (refers to R44 here)"
- note added: "isolated gate drivers; RET_ISO has no other connection on this board."

Commit message: Phase 2 done: footprints assigned and verified against IPC pads
- tools/gen_footprints.py -> lib/footprint_map.csv + lib/ac_psu.pretty (20 project footprints)
- tools/fpgeom.py: footprint pad loader and rigid fit; tools/check_footprints.py (+ pcbnew
  placement check), added to check_all.sh; reports/footprint_fit.csv for Phase 3 placement
- sch_builder: Footprint field from the map, deterministic UUIDs; all sheets regenerated
- kicad/fp-lib-table; STATUS.md (decisions, residuals, REF3025/C67 findings); Phase 3 prompt

Co-Authored-By: Claude Opus 5.5 <noreply@anthropic.com>
Parts:
- C15, C28: footprint (none) -> ac_psu:CP_Elec_6.3x7.7_EEEFTE221XAP
- C36, C41, C57, C58, C62, C65, C66, C67, C68: footprint (none) -> Capacitor_SMD:C_1206_3216Metric_Pad1.33x1.80mm_HandSolder
- C63: footprint (none) -> Capacitor_SMD:C_0603_1608Metric
- D1, D2, D6: footprint (none) -> ac_psu:D_SMA_AC
- D7: footprint (none) -> ac_psu:D_SOD-323_AC
- PWM1: footprint (none) -> Package_DIP:DIP-8-N6_W7.62mm
- R23, R24, R45, R47, R49: footprint (none) -> Resistor_SMD:R_1206_3216Metric
- R25, R26, R29, R31, R44: footprint (none) -> Resistor_SMD:R_0603_1608Metric
- R33, R34, R43: footprint (none) -> Resistor_SMD:R_1206_3216Metric_Pad1.30x1.75mm_HandSolder
- TR2: footprint (none) -> ac_psu:Transformer_EF20_2x5_P3.81mm
Changed lines of the file:
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@@
 			)
 		)
-		(property "Footprint" ""
+		(property "Footprint" "ac_psu:CP_Elec_6.3x7.7_EEEFTE221XAP"
 			(at 26.3652 38.1 0)
 			(effects
@@
 			)
 		)
-		(property "Footprint" ""
+		(property "Footprint" "Capacitor_SMD:C_1206_3216Metric_Pad1.33x1.80mm_HandSolder"
 			(at 36.5252 38.1 0)
 			(effects
@@
 			)
 		)
-		(property "Footprint" ""
+		(property "Footprint" "Capacitor_SMD:C_1206_3216Metric_Pad1.33x1.80mm_HandSolder"
 			(at 26.3652 55.88 0)
 			(effects
@@
 			)
 		)
-		(property "Footprint" ""
+		(property "Footprint" "Capacitor_SMD:C_1206_3216Metric_Pad1.33x1.80mm_HandSolder"
 			(at 36.5252 55.88 0)
 			(effects
@@
 			)
 		)
-		(property "Footprint" ""
+		(property "Footprint" "Capacitor_SMD:C_1206_3216Metric_Pad1.33x1.80mm_HandSolder"
 			(at 46.6852 55.88 0)
 			(effects
@@
 			)
 		)
-		(property "Footprint" ""
+		(property "Footprint" "Capacitor_SMD:C_1206_3216Metric_Pad1.33x1.80mm_HandSolder"
 			(at 87.9348 20.32 0)
 			(effects
@@
 			)
 		)
-		(property "Footprint" ""
+		(property "Footprint" "Resistor_SMD:R_1206_3216Metric_Pad1.30x1.75mm_HandSolder"
 			(at 79.502 25.4 0)
 			(effects
@@
 			)
 		)
-		(property "Footprint" ""
+		(property "Footprint" "Resistor_SMD:R_1206_3216Metric_Pad1.30x1.75mm_HandSolder"
 			(at 79.502 35.56 0)
 			(effects
@@
 			)
 		)
-		(property "Footprint" ""
+		(property "Footprint" "Resistor_SMD:R_1206_3216Metric_Pad1.30x1.75mm_HandSolder"
 			(at 79.502 45.72 0)
 			(effects
@@
 			)
 		)
-		(property "Footprint" ""
+		(property "Footprint" "Package_DIP:DIP-8-N6_W7.62mm"
 			(at 101.6 76.2 0)
 			(effects
@@
 			)
 		)
-		(property "Footprint" ""
+		(property "Footprint" "ac_psu:D_SOD-323_AC"
 			(at 58.42 69.85 0)
 			(effects
@@
 			)
 		)
-		(property "Footprint" ""
+		(property "Footprint" "Capacitor_SMD:C_1206_3216Metric_Pad1.33x1.80mm_HandSolder"
 			(at 67.0052 81.28 0)
 			(effects
@@
 			)
 		)
-		(property "Footprint" ""
+		(property "Footprint" "Capacitor_SMD:C_1206_3216Metric_Pad1.33x1.80mm_HandSolder"
 			(at 74.6252 81.28 0)
 			(effects
@@
 			)
 		)
-		(property "Footprint" ""
+		(property "Footprint" "Resistor_SMD:R_1206_3216Metric"
 			(at 112.522 24.13 0)
 			(effects
@@
 			)
 		)
-		(property "Footprint" ""
+		(property "Footprint" "Capacitor_SMD:C_1206_3216Metric_Pad1.33x1.80mm_HandSolder"
 			(at 125.4252 27.94 0)
 			(effects
@@
 			)
 		)
-		(property "Footprint" ""
+		(property "Footprint" "Resistor_SMD:R_1206_3216Metric"
 			(at 117.602 41.91 0)
 			(effects
@@
 			)
 		)
-		(property "Footprint" ""
+		(property "Footprint" "ac_psu:D_SMA_AC"
 			(at 119.38 54.61 0)
 			(effects
@@
 			)
 		)
-		(property "Footprint" ""
+		(property "Footprint" "Resistor_SMD:R_1206_3216Metric"
 			(at 130.302 86.36 0)
 			(effects
@@
 			)
 		)
-		(property "Footprint" ""
+		(property "Footprint" "Resistor_SMD:R_1206_3216Metric"
 			(at 137.922 86.36 0)
 			(effects
@@
 			)
 		)
-		(property "Footprint" ""
+		(property "Footprint" "ac_psu:D_SMA_AC"
 			(at 25.4 96.52 0)
 			(effects
@@
 			)
 		)
-		(property "Footprint" ""
+		(property "Footprint" "Resistor_SMD:R_0603_1608Metric"
 			(at 35.56 108.458 0)
 			(effects
@@
 			)
 		)
-		(property "Footprint" ""
+		(property "Footprint" "Resistor_SMD:R_0603_1608Metric"
 			(at 35.56 116.078 0)
 			(effects
@@
 			)
 		)
-		(property "Footprint" ""
+		(property "Footprint" "Capacitor_SMD:C_0603_1608Metric"
 			(at 49.8348 119.38 0)
 			(effects
@@
 			)
 		)
-		(property "Footprint" ""
+		(property "Footprint" "Resistor_SMD:R_0603_1608Metric"
 			(at 56.642 123.19 0)
 			(effects
@@
 			)
 		)
-		(property "Footprint" ""
+		(property "Footprint" "Resistor_SMD:R_0603_1608Metric"
 			(at 64.262 123.19 0)
 			(effects
@@
 			)
 		)
-		(property "Footprint" ""
+		(property "Footprint" "Resistor_SMD:R_0603_1608Metric"
 			(at 76.2 104.902 0)
 			(effects
@@
 			)
 		)
-		(property "Footprint" ""
+		(property "Footprint" "ac_psu:Transformer_EF20_2x5_P3.81mm"
 			(at 167.64 38.1 0)
 			(effects
@@
 			)
 		)
-		(property "Footprint" ""
+		(property "Footprint" "ac_psu:D_SMA_AC"
 			(at 182.88 40.64 0)
 			(effects
@@
 			)
 		)
-		(property "Footprint" ""
+		(property "Footprint" "Capacitor_SMD:C_1206_3216Metric_Pad1.33x1.80mm_HandSolder"
 			(at 194.0052 52.07 0)
 			(effects
@@
 			)
 		)
-		(property "Footprint" ""
+		(property "Footprint" "ac_psu:CP_Elec_6.3x7.7_EEEFTE221XAP"
 			(at 204.1652 52.07 0)
 			(effects
@@
 			)
 		)
-		(property "Footprint" ""
+		(property "Footprint" "Resistor_SMD:R_1206_3216Metric"
 			(at 215.138 48.26 0)
 			(effects

Commit message: v4 design fixes: RET_ISO->ISOGND, U11 INH->GND, C88/C89 on ADA2/ADA3, ADuM7701 RC compensation, R48 Kelvin split
Board frozen: kicad/ac_psu.kicad_pcb edited by one-shot pcbnew scripts tools/v4/fix_1..5
(apply_all.sh, reproducible from the tag's board); make_pcb.sh rebuilds the Proteus board from
tag proteus-conversion-complete into build/proteus/ (byte-identical, checked by regen_check).
Proteus comparisons apply exactly lib/v4_deviations.csv + lib/v4_copper.csv (tools/deviations.py,
wrappers compare_netlists_v4 / check_symbols_v4, deviation support in check_board,
check_footprints, gen_footprints, ipc356_diff, gerber_roundtrip). p2k submodule unchanged.
check_all: ALL CHECKS PASSED; DRC 0 shorts / 0 unconnected / 0 parity (+1 accepted courtyard
overlap C91/U5).

Co-Authored-By: Claude Opus 5.5 <noreply@anthropic.com>
Connections:
- net RET_ISO renamed ISOGND
Other:
- note added: "not connected to ISOGND although U8 and the gate drivers J4/J6/J8 return 20V_ISO_SEC on ISOGND)."
- note added: "v4: the isolated 20 V return is ISOGND (v3: the PDF's ISO_GND terminal was wired to RET_iso, net RET_ISO,"
- note removed: "The PDF's ISO_GND terminal is wired to RET_iso: net RET_ISO (not ISOGND). 20V_ISO_SEC feeds U8 (sheet 3) and the"
- note removed: "isolated gate drivers; RET_ISO has no other connection on this board."
Changed lines of the file:
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@@
 	)
 	(symbol
-		(lib_id "ac_psu:RET_ISO")
+		(lib_id "ac_psu:ISOGND")
 		(at 228.6 55.88 0)
 		(unit 1)
@@
 			)
 		)
-		(property "Value" "RET_ISO"
+		(property "Value" "ISOGND"
 			(at 228.6 59.69 0)
 			(effects
@@
 			)
 		)
-		(property "Description" "Power symbol for net \"RET_ISO\" (IPC net name)"
+		(property "Description" "Power symbol for net \"ISOGND\" (IPC net name)"
 			(at 228.6 55.88 0)
 			(effects
@@
 		)
 	)
-	(wire
-		(pts
-			(xy 228.6 55.88) (xy 228.6 53.34)
-		)
-		(stroke
-			(width 0)
-			(type default)
-		)
-	)
-	(symbol
-		(lib_id "ac_psu:PWR_FLAG")
-		(at 228.6 53.34 0)
-		(unit 1)
-		(exclude_from_sim no)
-		(in_bom yes)
-		(on_board yes)
-		(dnp no)
-		(property "Reference" "#FLG020"
-			(at 228.6 51.435 0)
-			(effects
-				(font
-					(size 1.27 1.27)
-				)
-				(hide yes)
-			)
-		)
-		(property "Value" "PWR_FLAG"
-			(at 228.6 49.53 0)
-			(effects
-				(font
-					(size 1.27 1.27)
-				)
-			)
-		)
-		(property "Footprint" ""
-			(at 228.6 53.34 0)
-			(effects
-				(font
-					(size 1.27 1.27)
-				)
-				(hide yes)
-			)
-		)
-		(property "Datasheet" ""
-			(at 228.6 53.34 0)
-			(effects
-				(font
-					(size 1.27 1.27)
-				)
-				(hide yes)
-			)
-		)
-		(property "Description" "Special symbol for telling ERC where power comes from"
-			(at 228.6 53.34 0)
-			(effects
-				(font
-					(size 1.27 1.27)
-				)
-				(hide yes)
-			)
-		)
-		(pin "1"
-		)
-		(instances
-			(project "ac_psu"
-				(path "/04fb09b4-531d-41de-805c-3ed4ed6dcfa8/e9f831a8-cac5-4226-8b62-2e91876072f4"
-					(reference "#FLG020")
-					(unit 1)
-				)
-			)
-		)
-	)
-	(text "The PDF's ISO_GND terminal is wired to RET_iso: net RET_ISO (not ISOGND). 20V_ISO_SEC feeds U8 (sheet 3) and the"
+	(text "v4: the isolated 20 V return is ISOGND (v3: the PDF's ISO_GND terminal was wired to RET_iso, net RET_ISO,"
 		(exclude_from_sim no)
 		(at 160.02 71.12 0)
@@
 		)
 	)
-	(text "isolated gate drivers; RET_ISO has no other connection on this board."
+	(text "not connected to ISOGND although U8 and the gate drivers J4/J6/J8 return 20V_ISO_SEC on ISOGND)."
 		(exclude_from_sim no)
 		(at 160.02 74.93 0)

Commit message: v4 clean-up: C67 drawn as a ceramic capacitor (symbol C), fix 7 copies its fields to the board
C67 (100 uF on 5V) sits on the same non-polar 1206 land pattern as C57/C58
with no polarity mark in Proteus; BOM part C15008 (100 uF 6.3 V X5R 1206).

Co-Authored-By: Claude Opus 5.5 <noreply@anthropic.com>
Claude-Session: https://claude.ai/code/session_01Am5hpeWpvZbzmHWspFiWJm
Parts:
- C67: symbol ac_psu:C_Polarized -> ac_psu:C
Other:
- note added: "C67: 100 uF ceramic (X5R 1206, non-polar land pattern like C57/C58; v4 clean-up, was drawn polarized)."
- note removed: "C67: IPC pin 1 is on GND (C28/C15 have pin 1 on the + rail) - check footprint polarity in Phase 2."
Changed lines of the file:
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@@
 	)
 	(symbol
-		(lib_id "ac_psu:C_Polarized")
+		(lib_id "ac_psu:C")
 		(at 25.4 52.07 0)
 		(unit 1)
@@
 			)
 		)
-		(property "Description" "Polarized capacitor, pin 1 = +"
+		(property "Description" "Unpolarized capacitor"
 			(at 25.4 52.07 0)
 			(effects
@@
 		)
 	)
-	(text "C67: IPC pin 1 is on GND (C28/C15 have pin 1 on the + rail) - check footprint polarity in Phase 2."
+	(text "C67: 100 uF ceramic (X5R 1206, non-polar land pattern like C57/C58; v4 clean-up, was drawn polarized)."
 		(exclude_from_sim no)
 		(at 25.4 147.32 0)
