File: kicad/01_afe.kicad_sch (KiCad schematic)
At the start: 48 parts, among them J5 PIN, Q1 C3M0065090D, Q2 C3M0065090D, Q3 C3M0065090D, Q4 C3M0065090D, U1 OPA2353UA

Commit message: v4 fix 11/12: measurement filters (reports/noise findings 1-5), AMC1306M05
Schematic (sheets 1/3/4/5/9): C95-C106 1n C0G across every 10k leg of the six
difference amplifiers (15.9 kHz tap-node filter), R7 1k -> 10k (U1B + leg
matched; ADA3 scaling changes), R18/R9 100R -> 8.2k with C88/C89 4.7n C0G and
new C107/C108 4.7n on ISOADA1/2 (4.1 kHz), C42/C2 1n -> 10n C0G (1.9 kHz DC
links), C109/C110 100n on REF_1V65/REF_1V65_ISO. R64/DAB series R unchanged
(L unknown; 25R per leg for 10 nH).
Board: fix 11 places the 16 caps (10 top beside their resistor, 6 bottom with
7 vias), renames six auto-named output nets, sets the values; fix 12 re-runs
fix 8's silk placement. DRC 293 (+1 silk), 0 shorts/unconnected/parity.
Deviation rows, v4_copper vias/areas, part map. Replay of fixes 1-12 on the
tag's board gives the board and edit log.
fab: C0G codes C307441/C1518204/C22400107, U4-U6 AMC1306M05DWVR (C701717,
+-50 mV, 4.9k R_IND, checked in SBAS734D), CPL 205 parts, stock for 5 boards
(AMC1306M05: 5 in stock). Noise report: CMTI 50 kV/us min correction.

Co-Authored-By: Claude Opus 5.5 <noreply@anthropic.com>
Claude-Session: https://claude.ai/code/session_01Am5hpeWpvZbzmHWspFiWJm
Parts:
- added C95, C96, C97, C98: 1n C0G, Capacitor_SMD:C_0402_1005Metric, symbol ac_psu:C
- R18, R9: value 100 -> 8.2k
- R7: value 1k -> 10k
Connections:
- net REF_1V65: now also C95.1, C97.1
- net at R8.1, R9.2, U1.7: now also C98.1
- net at R13.1, R21.2, U1.3 (+): now also C95.2
- net at R3.1, R8.2, U1.6 (-): now also C98.2
- net at R17.1, R18.2, U1.1: now also C96.1
- net at R16.1, R17.2, U1.2 (-): now also C96.2
- net at R6.1, R7.2, U1.5 (+): now also C97.2
Other:
- note added: "v4: R7 10k (v3 1k: + leg unmatched, common-mode gain ~0.033 - ADA3 was FILTER_INPUT vs GND); C95-C98 1n C0G across the 10k legs (15.9 kHz, tap-node HF filter); R18/R9 8.2k (v3 100R) with C88/C89 4.7n -> 4.1 kHz."
