File: kicad/04_dc_links.kicad_sch (KiCad schematic)
At the start: 0 parts

Commit message: Phase 1: sheets 6 (DAB) and 4 (DC links); diff_amp generalised for TLV316 blocks
Co-Authored-By: Claude Fable 5.1 <noreply@anthropic.com>
Parts:
- added C10, C59, C60, C7: 2n2, symbol ac_psu:C
- added C11, C12, C61, C72, C79, C8: SNAP_IN_35MM, symbol ac_psu:C_Polarized
- added C2, C42: 1n, symbol ac_psu:C
- added C27, C87: 100n, symbol ac_psu:C
- added PE8: PIN, symbol ac_psu:PIN
- added R1, R37, R38, R76: 10k, symbol ac_psu:R
- added R27, R28, R35, R36, R41, R42, R80, R81, R82, R83, R84, R85: 91K, symbol ac_psu:R
- added R39, R77: 8.2k, symbol ac_psu:R
- added R96, R97: 0R, symbol ac_psu:R
- added U14, U2: TLV316IDBVR, symbol ac_psu:TLV316IDBVR
Connections:
- new net: R38.1, R39.2, U14.1
- new net: R28.1, R36.2
- new net: R28.2, R42.1
- new net: R76.1, R77.2, U2.1
- new net: R76.2, R85.1, U2.4 (-)
- new net: R1.2, R82.1, U2.3 (+)
- new net: R83.1, R84.2
- new net: R35.1, R37.2, U14.3 (+)
- new net: R36.1, R38.2, U14.4 (-)
- new net: R27.2, R41.1
- new net: R80.1, R82.2
- new net: R80.2, R81.1
- new net: R84.1, R85.2
- new net: C10.2, C7.1, PE8.1
- new net: R27.1, R35.2
- new net 3V3_ISO: C87.2, U2.5 (V+)
- new net ADA1: C42.1, R39.1
- new net DC+: C11.1, C12.1, C7.2, C79.1, R41.2
- new net GND: C27.1, C42.2, R37.1, R96.1, U14.2 (V-)
- new net ISOADA3: C2.1, R77.1
- new net ISODC+: C59.2, C61.1, C72.1, C8.1, R81.2
- new net ISOGND: C2.2, C87.1, R1.1, R97.1, U2.2 (V-)
- new net ISOPGND: C60.1, C61.2, C72.2, C8.2, R83.2, R97.2
- new net PE5: C59.1, C60.2
- new net PGND: C10.1, C11.2, C12.2, C79.2, R42.2, R96.2
- new net VCC: C27.2, U14.5 (V+)
Other:
- note added: "Measurement connections (0 R)"
- note added: "Primary and isolated DC links. PE8 terminal is on this sheet; PE5 is on sheet 5."
- note added: "U14: (DC+ - PGND) / 3 x 91K, output -> ADA1 (sheet 9). DC- in the PDF = GND."
- note added: "U2: (ISODC+ - ISOPGND) / 3 x 91K, output -> ISOADA3 (J11)."

Commit message: Phase 2 done: footprints assigned and verified against IPC pads
- tools/gen_footprints.py -> lib/footprint_map.csv + lib/ac_psu.pretty (20 project footprints)
- tools/fpgeom.py: footprint pad loader and rigid fit; tools/check_footprints.py (+ pcbnew
  placement check), added to check_all.sh; reports/footprint_fit.csv for Phase 3 placement
- sch_builder: Footprint field from the map, deterministic UUIDs; all sheets regenerated
- kicad/fp-lib-table; STATUS.md (decisions, residuals, REF3025/C67 findings); Phase 3 prompt

Co-Authored-By: Claude Opus 5.5 <noreply@anthropic.com>
Parts:
- C10, C59, C60, C7: footprint (none) -> Capacitor_THT:C_Disc_D12.5mm_W5.0mm_P7.50mm
- C11, C12, C61, C72, C79, C8: footprint (none) -> Capacitor_THT:CP_Radial_D35.0mm_P10.00mm_SnapIn
- C2, C27, C42, C87: footprint (none) -> Capacitor_SMD:C_0402_1005Metric
- PE8: footprint (none) -> ac_psu:Terminal_D3.05mm_Drill1.52mm
- R1, R37, R38, R39, R76, R77: footprint (none) -> Resistor_SMD:R_0402_1005Metric
- R27, R28, R35, R36, R41, R42, R80, R81, R82, R83, R84, R85, R96, R97: footprint (none) -> Resistor_SMD:R_1206_3216Metric_Pad1.30x1.75mm_HandSolder
- U14, U2: footprint (none) -> ac_psu:SOT-23-5_TLV316
Changed lines of the file:
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@@
 			)
 		)
-		(property "Footprint" ""
+		(property "Footprint" "Capacitor_THT:CP_Radial_D35.0mm_P10.00mm_SnapIn"
 			(at 26.3652 49.53 0)
 			(effects
@@
 			)
 		)
-		(property "Footprint" ""
+		(property "Footprint" "Capacitor_THT:CP_Radial_D35.0mm_P10.00mm_SnapIn"
 			(at 46.6852 49.53 0)
 			(effects
@@
 			)
 		)
-		(property "Footprint" ""
+		(property "Footprint" "Capacitor_THT:CP_Radial_D35.0mm_P10.00mm_SnapIn"
 			(at 67.0052 49.53 0)
 			(effects
@@
 			)
 		)
-		(property "Footprint" ""
+		(property "Footprint" "Capacitor_THT:C_Disc_D12.5mm_W5.0mm_P7.50mm"
 			(at 80.3148 34.29 0)
 			(effects
@@
 			)
 		)
-		(property "Footprint" ""
+		(property "Footprint" "Capacitor_THT:C_Disc_D12.5mm_W5.0mm_P7.50mm"
 			(at 80.3148 49.53 0)
 			(effects
@@
 			)
 		)
-		(property "Footprint" ""
+		(property "Footprint" "ac_psu:Terminal_D3.05mm_Drill1.52mm"
 			(at 88.9 50.8 0)
 			(effects
@@
 			)
 		)
-		(property "Footprint" ""
+		(property "Footprint" "Capacitor_THT:CP_Radial_D35.0mm_P10.00mm_SnapIn"
 			(at 26.3652 125.73 0)
 			(effects
@@
 			)
 		)
-		(property "Footprint" ""
+		(property "Footprint" "Capacitor_THT:CP_Radial_D35.0mm_P10.00mm_SnapIn"
 			(at 46.6852 125.73 0)
 			(effects
@@
 			)
 		)
-		(property "Footprint" ""
+		(property "Footprint" "Capacitor_THT:CP_Radial_D35.0mm_P10.00mm_SnapIn"
 			(at 67.0052 125.73 0)
 			(effects
@@
 			)
 		)
-		(property "Footprint" ""
+		(property "Footprint" "Capacitor_THT:C_Disc_D12.5mm_W5.0mm_P7.50mm"
 			(at 80.3148 110.49 0)
 			(effects
@@
 			)
 		)
-		(property "Footprint" ""
+		(property "Footprint" "Capacitor_THT:C_Disc_D12.5mm_W5.0mm_P7.50mm"
 			(at 80.3148 125.73 0)
 			(effects
@@
 			)
 		)
-		(property "Footprint" ""
+		(property "Footprint" "Resistor_SMD:R_1206_3216Metric_Pad1.30x1.75mm_HandSolder"
 			(at 50.8 158.242 0)
 			(effects
@@
 			)
 		)
-		(property "Footprint" ""
+		(property "Footprint" "Resistor_SMD:R_1206_3216Metric_Pad1.30x1.75mm_HandSolder"
 			(at 50.8 168.402 0)
 			(effects
@@
 			)
 		)
-		(property "Footprint" ""
+		(property "Footprint" "Resistor_SMD:R_1206_3216Metric_Pad1.30x1.75mm_HandSolder"
 			(at 199.898 45.72 0)
 			(effects
@@
 			)
 		)
-		(property "Footprint" ""
+		(property "Footprint" "Resistor_SMD:R_1206_3216Metric_Pad1.30x1.75mm_HandSolder"
 			(at 199.898 55.88 0)
 			(effects
@@
 			)
 		)
-		(property "Footprint" ""
+		(property "Footprint" "Resistor_SMD:R_1206_3216Metric_Pad1.30x1.75mm_HandSolder"
 			(at 199.898 66.04 0)
 			(effects
@@
 			)
 		)
-		(property "Footprint" ""
+		(property "Footprint" "Resistor_SMD:R_1206_3216Metric_Pad1.30x1.75mm_HandSolder"
 			(at 192.278 45.72 0)
 			(effects
@@
 			)
 		)
-		(property "Footprint" ""
+		(property "Footprint" "Resistor_SMD:R_1206_3216Metric_Pad1.30x1.75mm_HandSolder"
 			(at 192.278 55.88 0)
 			(effects
@@
 			)
 		)
-		(property "Footprint" ""
+		(property "Footprint" "Resistor_SMD:R_1206_3216Metric_Pad1.30x1.75mm_HandSolder"
 			(at 192.278 66.04 0)
 			(effects
@@
 			)
 		)
-		(property "Footprint" ""
+		(property "Footprint" "ac_psu:SOT-23-5_TLV316"
 			(at 215.9 81.28 0)
 			(effects
@@
 			)
 		)
-		(property "Footprint" ""
+		(property "Footprint" "Resistor_SMD:R_0402_1005Metric"
 			(at 206.502 66.04 0)
 			(effects
@@
 			)
 		)
-		(property "Footprint" ""
+		(property "Footprint" "Resistor_SMD:R_0402_1005Metric"
 			(at 236.22 74.422 0)
 			(effects
@@
 			)
 		)
-		(property "Footprint" ""
+		(property "Footprint" "Capacitor_SMD:C_0402_1005Metric"
 			(at 243.5352 87.63 0)
 			(effects
@@
 			)
 		)
-		(property "Footprint" ""
+		(property "Footprint" "Resistor_SMD:R_0402_1005Metric"
 			(at 218.44 82.042 0)
 			(effects
@@
 			)
 		)
-		(property "Footprint" ""
+		(property "Footprint" "Resistor_SMD:R_1206_3216Metric_Pad1.30x1.75mm_HandSolder"
 			(at 199.898 121.92 0)
 			(effects
@@
 			)
 		)
-		(property "Footprint" ""
+		(property "Footprint" "Resistor_SMD:R_1206_3216Metric_Pad1.30x1.75mm_HandSolder"
 			(at 199.898 132.08 0)
 			(effects
@@
 			)
 		)
-		(property "Footprint" ""
+		(property "Footprint" "Resistor_SMD:R_1206_3216Metric_Pad1.30x1.75mm_HandSolder"
 			(at 199.898 142.24 0)
 			(effects
@@
 			)
 		)
-		(property "Footprint" ""
+		(property "Footprint" "Resistor_SMD:R_1206_3216Metric_Pad1.30x1.75mm_HandSolder"
 			(at 192.278 121.92 0)
 			(effects
@@
 			)
 		)
-		(property "Footprint" ""
+		(property "Footprint" "Resistor_SMD:R_1206_3216Metric_Pad1.30x1.75mm_HandSolder"
 			(at 192.278 132.08 0)
 			(effects
@@
 			)
 		)
-		(property "Footprint" ""
+		(property "Footprint" "Resistor_SMD:R_1206_3216Metric_Pad1.30x1.75mm_HandSolder"
 			(at 192.278 142.24 0)
 			(effects
@@
 			)
 		)
-		(property "Footprint" ""
+		(property "Footprint" "ac_psu:SOT-23-5_TLV316"
 			(at 215.9 157.48 0)
 			(effects
@@
 			)
 		)
-		(property "Footprint" ""
+		(property "Footprint" "Resistor_SMD:R_0402_1005Metric"
 			(at 206.502 142.24 0)
 			(effects
@@
 			)
 		)
-		(property "Footprint" ""
+		(property "Footprint" "Resistor_SMD:R_0402_1005Metric"
 			(at 236.22 150.622 0)
 			(effects
@@
 			)
 		)
-		(property "Footprint" ""
+		(property "Footprint" "Capacitor_SMD:C_0402_1005Metric"
 			(at 243.5352 163.83 0)
 			(effects
@@
 			)
 		)
-		(property "Footprint" ""
+		(property "Footprint" "Resistor_SMD:R_0402_1005Metric"
 			(at 218.44 158.242 0)
 			(effects
@@
 			)
 		)
-		(property "Footprint" ""
+		(property "Footprint" "Capacitor_SMD:C_0402_1005Metric"
 			(at 265.7348 52.07 0)
 			(effects
@@
 			)
 		)
-		(property "Footprint" ""
+		(property "Footprint" "Capacitor_SMD:C_0402_1005Metric"
 			(at 265.7348 128.27 0)
 			(effects

Commit message: Phase 3 done: PCB rebuilt from the Proteus gerbers with nets and zones
tools/make_pcb.sh regenerates kicad/ac_psu.kicad_pcb (byte-reproducible):
build_pcb.py (footprints with nets and symbol links at the Proteus
positions, outline, mounting holes, rules), gerber_to_tracks.py (4052
tracks, 173 vias; pour edge strokes recognised and skipped),
assign_nets.py (union-find over copper, 0 shorts/orphans/opens with
pours), pours_to_zones.py (79 zones = Proteus pour copper incl. holes).

New checks in check_all.sh: check_board.py (pads/holes/vias vs IPC),
assign_nets.py --check (after zone fill), drc.py (0 shorts, 0
unconnected, 0 parity issues; courtyard overlaps accepted).

Footprints (user decision): Proteus pad sizes for the headers, TSSOP,
SOT-23(-5), SOIC-16W packages whose KiCad pads shorted/violated
clearance; Proteus pads and drills for TO-247, VXO7805, P27.5 film and
snap-in caps; tighter courtyards for IPC-built footprints.

Co-Authored-By: Claude Opus 5.5 <noreply@anthropic.com>
Parts:
- C11, C12, C61, C72, C79, C8: footprint Capacitor_THT:CP_Radial_D35.0mm_P10.00mm_SnapIn -> ac_psu:CP_Radial_D35.0mm_P10.00mm_SnapIn_Proteus
Changed lines of the file:
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@@
 			)
 		)
-		(property "Footprint" "Capacitor_THT:CP_Radial_D35.0mm_P10.00mm_SnapIn"
+		(property "Footprint" "ac_psu:CP_Radial_D35.0mm_P10.00mm_SnapIn_Proteus"
 			(at 26.3652 49.53 0)
 			(effects
@@
 			)
 		)
-		(property "Footprint" "Capacitor_THT:CP_Radial_D35.0mm_P10.00mm_SnapIn"
+		(property "Footprint" "ac_psu:CP_Radial_D35.0mm_P10.00mm_SnapIn_Proteus"
 			(at 46.6852 49.53 0)
 			(effects
@@
 			)
 		)
-		(property "Footprint" "Capacitor_THT:CP_Radial_D35.0mm_P10.00mm_SnapIn"
+		(property "Footprint" "ac_psu:CP_Radial_D35.0mm_P10.00mm_SnapIn_Proteus"
 			(at 67.0052 49.53 0)
 			(effects
@@
 			)
 		)
-		(property "Footprint" "Capacitor_THT:CP_Radial_D35.0mm_P10.00mm_SnapIn"
+		(property "Footprint" "ac_psu:CP_Radial_D35.0mm_P10.00mm_SnapIn_Proteus"
 			(at 26.3652 125.73 0)
 			(effects
@@
 			)
 		)
-		(property "Footprint" "Capacitor_THT:CP_Radial_D35.0mm_P10.00mm_SnapIn"
+		(property "Footprint" "ac_psu:CP_Radial_D35.0mm_P10.00mm_SnapIn_Proteus"
 			(at 46.6852 125.73 0)
 			(effects
@@
 			)
 		)
-		(property "Footprint" "Capacitor_THT:CP_Radial_D35.0mm_P10.00mm_SnapIn"
+		(property "Footprint" "ac_psu:CP_Radial_D35.0mm_P10.00mm_SnapIn_Proteus"
 			(at 67.0052 125.73 0)
 			(effects

Commit message: v4 fix 11/12: measurement filters (reports/noise findings 1-5), AMC1306M05
Schematic (sheets 1/3/4/5/9): C95-C106 1n C0G across every 10k leg of the six
difference amplifiers (15.9 kHz tap-node filter), R7 1k -> 10k (U1B + leg
matched; ADA3 scaling changes), R18/R9 100R -> 8.2k with C88/C89 4.7n C0G and
new C107/C108 4.7n on ISOADA1/2 (4.1 kHz), C42/C2 1n -> 10n C0G (1.9 kHz DC
links), C109/C110 100n on REF_1V65/REF_1V65_ISO. R64/DAB series R unchanged
(L unknown; 25R per leg for 10 nH).
Board: fix 11 places the 16 caps (10 top beside their resistor, 6 bottom with
7 vias), renames six auto-named output nets, sets the values; fix 12 re-runs
fix 8's silk placement. DRC 293 (+1 silk), 0 shorts/unconnected/parity.
Deviation rows, v4_copper vias/areas, part map. Replay of fixes 1-12 on the
tag's board gives the board and edit log.
fab: C0G codes C307441/C1518204/C22400107, U4-U6 AMC1306M05DWVR (C701717,
+-50 mV, 4.9k R_IND, checked in SBAS734D), CPL 205 parts, stock for 5 boards
(AMC1306M05: 5 in stock). Noise report: CMTI 50 kV/us min correction.

Co-Authored-By: Claude Opus 5.5 <noreply@anthropic.com>
Claude-Session: https://claude.ai/code/session_01Am5hpeWpvZbzmHWspFiWJm
Parts:
- added C100, C101, C102, C99: 1n C0G, Capacitor_SMD:C_0402_1005Metric, symbol ac_psu:C
- C2, C42: value 1n -> 10n C0G
Connections:
- net GND: now also C99.1
- net ISOGND: now also C101.1
- net at R38.1, R39.2, U14.1: now also C100.1
- net at R36.1, R38.2, U14.4 (-): now also C100.2
- net at R35.1, R37.2, U14.3 (+): now also C99.2
- net at R1.2, R82.1, U2.3 (+): now also C101.2
- net at R76.2, R85.1, U2.4 (-): now also C102.2
- net at R76.1, R77.2, U2.1: now also C102.1
Other:
- note added: "v4: C99-C102 1n C0G across the 10k legs (15.9 kHz); C42/C2 10n (v3 1n) -> 8.2k/10n = 1.9 kHz DC-link filters."
