File: kicad/05_vsi.kicad_sch (KiCad schematic)
At the start: 0 parts

Commit message: Phase 1: sheet 5 (VSI); diff_amp shared helper, layout fixes on sheets 1/8
Co-Authored-By: Claude Fable 5.1 <noreply@anthropic.com>
Parts:
- added ACOUT1, ACOUT2, INU_OUT2, J10, J7, J9, PE5, PE6, PE7: PIN, symbol ac_psu:PIN
- added C29, C30, C31, C32: 2n2, symbol ac_psu:C
- added C33, C34: 7u, symbol ac_psu:C
- added C38, C56: 100n, symbol ac_psu:C
- added CM3: WE-CMBNC, symbol ac_psu:WE-CMBNC
- added Q5, Q6, Q7, Q8: C3M0065090D, symbol ac_psu:C3M0065090D
- added R256, R60, R61, R62, R63, R65, R66, R67, R68, R69, R70, R71: 91K, symbol ac_psu:R
- added R46, R51, R52, R53: 10k, symbol ac_psu:R
- added R54, R56: 8.2k, symbol ac_psu:R
- added R79: SLA-12VDC-SL-A, symbol ac_psu:SLA-12VDC-SL-A
- added R91: FKK5R0020FE-TR, symbol ac_psu:FKK5R0020FE-TR
- added U7: OPA2353UA, symbol ac_psu:OPA2353UA
Connections:
- new net: R46.2, R67.1, U7.5 (+)
- new net: R51.2, R68.1, U7.6 (-)
- new net: R51.1, R56.2, U7.7
- new net: R62.1, R63.2
- new net: R69.2, R70.1
- new net: R53.1, R54.2, U7.1
- new net: R256.1, R53.2, U7.2 (-)
- new net: R52.2, R71.1, U7.3 (+)
- new net: R66.1, R67.2
- new net: R65.1, R66.2
- new net: R61.1, R71.2
- new net: R60.1, R61.2
- new net: R68.2, R69.1
- new net: R256.2, R63.1
- new net: J7.1, R91.4
- new net 20V_ISO_SEC: R79.6 (COIL_2)
- new net 3V3_ISO: C38.2, C56.2, U7.8 (V+)
- new net AC_OUT_1: ACOUT1.1, R70.2, R79.3 (NO)
- new net AC_OUT_2: ACOUT2.1, C31.2, C34.2, CM3.4, R65.2
- new net AFE_RELAY: C32.2, C34.1, CM3.3, R79.1 (COM_1)
- new net INDUCTOR_OUTPUT: C29.2, C33.2, CM3.1, J9.1, R62.2
- new net INU_FILTER_INPUT: C30.2, C33.1, CM3.2, J10.1, R60.2
- new net INU_SHUNT1: R91.2
- new net INU_SHUNT2: R91.1
- new net ISOADA1: R54.1
- new net ISOADA2: R56.1
- new net ISODC+: Q5.2 (D), Q7.2 (D)
- new net ISOGND: C38.1, C56.1, U7.4 (V-)
- new net ISOPGND: Q6.3 (S), Q8.3 (S)
- new net PE5: PE5.1
- new net PE6: C29.1, C30.1, PE6.1
- new net PE7: C31.1, C32.1, PE7.1
- new net Q5_G: Q5.1 (G)
- new net Q5_S: INU_OUT2.1, Q5.3 (S), Q6.2 (D)
- new net Q6_G: Q6.1 (G)
- new net Q7_G: Q7.1 (G)
- new net Q7_S: Q7.3 (S), Q8.2 (D), R91.3
- new net Q8_G: Q8.1 (G)
- new net REF_1V65_ISO: R46.1, R52.1
- new net RELAY_DRIVE_ISO: R79.2 (COIL_1)
- no-connect marks 0 -> 1
Other:
- note added: "1/2 = INU_SHUNT2/INU_SHUNT1 sense -> U4 (sheet 10)."
- note added: "Output filter between the inverter (J9/J10, inductor on J7/J9 off-board) and ACOUT1/ACOUT2; R79 connects the output."
- note added: "PDF note: IKZ50N65EH5XKSA1 (alternative switch)."
- note added: "R91 2 mOhm shunt: 3 = Q7/Q8 midpoint, 4 = inductor_input -> J7,"
- note added: "U7:A measures the filter voltage (INU_FILTER_INPUT - INDUCTOR_OUTPUT) around REF_1V65_ISO -> ISOADA1."
- note added: "U7:B measures the output voltage (AC_OUT_2 - AC_OUT_1) around REF_1V65_ISO -> ISOADA2."
- note added: "VSI half bridges on the isolated DC link. Q6/Q8 sources are ISOPGND (Proteus: Q6_S / Q8_S at J6)."

Commit message: Phase 2 done: footprints assigned and verified against IPC pads
- tools/gen_footprints.py -> lib/footprint_map.csv + lib/ac_psu.pretty (20 project footprints)
- tools/fpgeom.py: footprint pad loader and rigid fit; tools/check_footprints.py (+ pcbnew
  placement check), added to check_all.sh; reports/footprint_fit.csv for Phase 3 placement
- sch_builder: Footprint field from the map, deterministic UUIDs; all sheets regenerated
- kicad/fp-lib-table; STATUS.md (decisions, residuals, REF3025/C67 findings); Phase 3 prompt

Co-Authored-By: Claude Opus 5.5 <noreply@anthropic.com>
Parts:
- ACOUT1, ACOUT2: footprint (none) -> ac_psu:Terminal_2x1_P5.00mm_D2.0mm_Drill1.4mm
- C29, C30, C31, C32: footprint (none) -> Capacitor_THT:C_Disc_D12.5mm_W5.0mm_P7.50mm
- C33, C34: footprint (none) -> Capacitor_THT:C_Rect_L33.0mm_W20.0mm_P27.50mm_MKS4
- C38, C56: footprint (none) -> Capacitor_SMD:C_0402_1005Metric
- CM3: footprint (none) -> ac_psu:L_CommonMode_WE-CMBNC
- INU_OUT2, J10, J7, J9: footprint (none) -> ac_psu:Terminal_D4.0mm_Drill2.55mm
- PE5, PE6, PE7: footprint (none) -> ac_psu:Terminal_D4.0mm_Drill3.0mm
- Q5, Q6, Q7, Q8: footprint (none) -> Package_TO_SOT_THT:TO-247-3_Vertical
- R256, R60, R61, R62, R63, R65, R66, R67, R68, R69, R70, R71: footprint (none) -> Resistor_SMD:R_1206_3216Metric_Pad1.30x1.75mm_HandSolder
- R46, R51, R52, R53, R54, R56: footprint (none) -> Resistor_SMD:R_0402_1005Metric
- R79: footprint (none) -> ac_psu:Relay_SLA-12VDC-SL-A
- R91: footprint (none) -> ac_psu:R_Shunt_FKK5R0020FE
- U7: footprint (none) -> Package_SO:TSSOP-8_3x3mm_P0.65mm
Changed lines of the file:
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@@
 			)
 		)
-		(property "Footprint" ""
+		(property "Footprint" "Package_TO_SOT_THT:TO-247-3_Vertical"
 			(at 55.88 48.26 0)
 			(effects
@@
 			)
 		)
-		(property "Footprint" ""
+		(property "Footprint" "Package_TO_SOT_THT:TO-247-3_Vertical"
 			(at 55.88 86.36 0)
 			(effects
@@
 			)
 		)
-		(property "Footprint" ""
+		(property "Footprint" "ac_psu:Terminal_D4.0mm_Drill2.55mm"
 			(at 68.58 74.93 0)
 			(effects
@@
 			)
 		)
-		(property "Footprint" ""
+		(property "Footprint" "Package_TO_SOT_THT:TO-247-3_Vertical"
 			(at 106.68 48.26 0)
 			(effects
@@
 			)
 		)
-		(property "Footprint" ""
+		(property "Footprint" "Package_TO_SOT_THT:TO-247-3_Vertical"
 			(at 106.68 86.36 0)
 			(effects
@@
 			)
 		)
-		(property "Footprint" ""
+		(property "Footprint" "ac_psu:R_Shunt_FKK5R0020FE"
 			(at 148.082 45.72 0)
 			(effects
@@
 			)
 		)
-		(property "Footprint" ""
+		(property "Footprint" "ac_psu:Terminal_D4.0mm_Drill2.55mm"
 			(at 160.02 53.34 0)
 			(effects
@@
 			)
 		)
-		(property "Footprint" ""
+		(property "Footprint" "ac_psu:Terminal_D4.0mm_Drill2.55mm"
 			(at 220.98 50.8 0)
 			(effects
@@
 			)
 		)
-		(property "Footprint" ""
+		(property "Footprint" "ac_psu:Terminal_D4.0mm_Drill2.55mm"
 			(at 210.82 60.96 0)
 			(effects
@@
 			)
 		)
-		(property "Footprint" ""
+		(property "Footprint" "Capacitor_THT:C_Disc_D12.5mm_W5.0mm_P7.50mm"
 			(at 224.4852 46.99 0)
 			(effects
@@
 			)
 		)
-		(property "Footprint" ""
+		(property "Footprint" "Capacitor_THT:C_Disc_D12.5mm_W5.0mm_P7.50mm"
 			(at 222.5548 64.77 0)
 			(effects
@@
 			)
 		)
-		(property "Footprint" ""
+		(property "Footprint" "Capacitor_THT:C_Rect_L33.0mm_W20.0mm_P27.50mm_MKS4"
 			(at 232.1052 59.69 0)
 			(effects
@@
 			)
 		)
-		(property "Footprint" ""
+		(property "Footprint" "ac_psu:L_CommonMode_WE-CMBNC"
 			(at 241.3 62.23 0)
 			(effects
@@
 			)
 		)
-		(property "Footprint" ""
+		(property "Footprint" "Capacitor_THT:C_Disc_D12.5mm_W5.0mm_P7.50mm"
 			(at 254.9652 46.99 0)
 			(effects
@@
 			)
 		)
-		(property "Footprint" ""
+		(property "Footprint" "Capacitor_THT:C_Disc_D12.5mm_W5.0mm_P7.50mm"
 			(at 253.0348 64.77 0)
 			(effects
@@
 			)
 		)
-		(property "Footprint" ""
+		(property "Footprint" "Capacitor_THT:C_Rect_L33.0mm_W20.0mm_P27.50mm_MKS4"
 			(at 262.5852 59.69 0)
 			(effects
@@
 			)
 		)
-		(property "Footprint" ""
+		(property "Footprint" "ac_psu:Relay_SLA-12VDC-SL-A"
 			(at 281.94 33.02 0)
 			(effects
@@
 			)
 		)
-		(property "Footprint" ""
+		(property "Footprint" "ac_psu:Terminal_2x1_P5.00mm_D2.0mm_Drill1.4mm"
 			(at 314.96 35.56 0)
 			(effects
@@
 			)
 		)
-		(property "Footprint" ""
+		(property "Footprint" "ac_psu:Terminal_2x1_P5.00mm_D2.0mm_Drill1.4mm"
 			(at 314.96 66.04 0)
 			(effects
@@
 			)
 		)
-		(property "Footprint" ""
+		(property "Footprint" "Resistor_SMD:R_1206_3216Metric_Pad1.30x1.75mm_HandSolder"
 			(at 210.058 76.2 0)
 			(effects
@@
 			)
 		)
-		(property "Footprint" ""
+		(property "Footprint" "Resistor_SMD:R_1206_3216Metric_Pad1.30x1.75mm_HandSolder"
 			(at 210.058 86.36 0)
 			(effects
@@
 			)
 		)
-		(property "Footprint" ""
+		(property "Footprint" "Resistor_SMD:R_1206_3216Metric_Pad1.30x1.75mm_HandSolder"
 			(at 210.058 96.52 0)
 			(effects
@@
 			)
 		)
-		(property "Footprint" ""
+		(property "Footprint" "Resistor_SMD:R_1206_3216Metric_Pad1.30x1.75mm_HandSolder"
 			(at 202.438 76.2 0)
 			(effects
@@
 			)
 		)
-		(property "Footprint" ""
+		(property "Footprint" "Resistor_SMD:R_1206_3216Metric_Pad1.30x1.75mm_HandSolder"
 			(at 202.438 86.36 0)
 			(effects
@@
 			)
 		)
-		(property "Footprint" ""
+		(property "Footprint" "Resistor_SMD:R_1206_3216Metric_Pad1.30x1.75mm_HandSolder"
 			(at 202.438 96.52 0)
 			(effects
@@
 			)
 		)
-		(property "Footprint" ""
+		(property "Footprint" "Package_SO:TSSOP-8_3x3mm_P0.65mm"
 			(at 228.6 106.68 0)
 			(effects
@@
 			)
 		)
-		(property "Footprint" ""
+		(property "Footprint" "Resistor_SMD:R_0402_1005Metric"
 			(at 216.662 96.52 0)
 			(effects
@@
 			)
 		)
-		(property "Footprint" ""
+		(property "Footprint" "Resistor_SMD:R_0402_1005Metric"
 			(at 246.38 104.902 0)
 			(effects
@@
 			)
 		)
-		(property "Footprint" ""
+		(property "Footprint" "Resistor_SMD:R_0402_1005Metric"
 			(at 228.6 112.522 0)
 			(effects
@@
 			)
 		)
-		(property "Footprint" ""
+		(property "Footprint" "Resistor_SMD:R_1206_3216Metric_Pad1.30x1.75mm_HandSolder"
 			(at 309.118 121.92 0)
 			(effects
@@
 			)
 		)
-		(property "Footprint" ""
+		(property "Footprint" "Resistor_SMD:R_1206_3216Metric_Pad1.30x1.75mm_HandSolder"
 			(at 309.118 132.08 0)
 			(effects
@@
 			)
 		)
-		(property "Footprint" ""
+		(property "Footprint" "Resistor_SMD:R_1206_3216Metric_Pad1.30x1.75mm_HandSolder"
 			(at 309.118 142.24 0)
 			(effects
@@
 			)
 		)
-		(property "Footprint" ""
+		(property "Footprint" "Resistor_SMD:R_1206_3216Metric_Pad1.30x1.75mm_HandSolder"
 			(at 301.498 121.92 0)
 			(effects
@@
 			)
 		)
-		(property "Footprint" ""
+		(property "Footprint" "Resistor_SMD:R_1206_3216Metric_Pad1.30x1.75mm_HandSolder"
 			(at 301.498 132.08 0)
 			(effects
@@
 			)
 		)
-		(property "Footprint" ""
+		(property "Footprint" "Resistor_SMD:R_1206_3216Metric_Pad1.30x1.75mm_HandSolder"
 			(at 301.498 142.24 0)
 			(effects
@@
 			)
 		)
-		(property "Footprint" ""
+		(property "Footprint" "Package_SO:TSSOP-8_3x3mm_P0.65mm"
 			(at 327.66 152.4 0)
 			(effects
@@
 			)
 		)
-		(property "Footprint" ""
+		(property "Footprint" "Resistor_SMD:R_0402_1005Metric"
 			(at 315.722 142.24 0)
 			(effects
@@
 			)
 		)
-		(property "Footprint" ""
+		(property "Footprint" "Resistor_SMD:R_0402_1005Metric"
 			(at 345.44 150.622 0)
 			(effects
@@
 			)
 		)
-		(property "Footprint" ""
+		(property "Footprint" "Resistor_SMD:R_0402_1005Metric"
 			(at 327.66 158.242 0)
 			(effects
@@
 			)
 		)
-		(property "Footprint" ""
+		(property "Footprint" "Package_SO:TSSOP-8_3x3mm_P0.65mm"
 			(at 38.1 152.4 0)
 			(effects
@@
 			)
 		)
-		(property "Footprint" ""
+		(property "Footprint" "Capacitor_SMD:C_0402_1005Metric"
 			(at 54.9148 148.59 0)
 			(effects
@@
 			)
 		)
-		(property "Footprint" ""
+		(property "Footprint" "Capacitor_SMD:C_0402_1005Metric"
 			(at 65.0748 148.59 0)
 			(effects
@@
 			)
 		)
-		(property "Footprint" ""
+		(property "Footprint" "ac_psu:Terminal_D4.0mm_Drill3.0mm"
 			(at 20.32 190.5 0)
 			(effects
@@
 			)
 		)
-		(property "Footprint" ""
+		(property "Footprint" "ac_psu:Terminal_D4.0mm_Drill3.0mm"
 			(at 30.48 190.5 0)
 			(effects
@@
 			)
 		)
-		(property "Footprint" ""
+		(property "Footprint" "ac_psu:Terminal_D4.0mm_Drill3.0mm"
 			(at 40.64 190.5 0)
 			(effects

Commit message: Phase 3 done: PCB rebuilt from the Proteus gerbers with nets and zones
tools/make_pcb.sh regenerates kicad/ac_psu.kicad_pcb (byte-reproducible):
build_pcb.py (footprints with nets and symbol links at the Proteus
positions, outline, mounting holes, rules), gerber_to_tracks.py (4052
tracks, 173 vias; pour edge strokes recognised and skipped),
assign_nets.py (union-find over copper, 0 shorts/orphans/opens with
pours), pours_to_zones.py (79 zones = Proteus pour copper incl. holes).

New checks in check_all.sh: check_board.py (pads/holes/vias vs IPC),
assign_nets.py --check (after zone fill), drc.py (0 shorts, 0
unconnected, 0 parity issues; courtyard overlaps accepted).

Footprints (user decision): Proteus pad sizes for the headers, TSSOP,
SOT-23(-5), SOIC-16W packages whose KiCad pads shorted/violated
clearance; Proteus pads and drills for TO-247, VXO7805, P27.5 film and
snap-in caps; tighter courtyards for IPC-built footprints.

Co-Authored-By: Claude Opus 5.5 <noreply@anthropic.com>
Parts:
- C33, C34: footprint Capacitor_THT:C_Rect_L33.0mm_W20.0mm_P27.50mm_MKS4 -> ac_psu:C_Rect_L33.0mm_W20.0mm_P27.50mm_MKS4_Proteus
- Q5, Q6, Q7, Q8: footprint Package_TO_SOT_THT:TO-247-3_Vertical -> ac_psu:TO-247-3_Vertical_Proteus
- U7: footprint Package_SO:TSSOP-8_3x3mm_P0.65mm -> ac_psu:TSSOP-8_3x3mm_P0.65mm_Proteus
Changed lines of the file:
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@@
 			)
 		)
-		(property "Footprint" "Package_TO_SOT_THT:TO-247-3_Vertical"
+		(property "Footprint" "ac_psu:TO-247-3_Vertical_Proteus"
 			(at 55.88 48.26 0)
 			(effects
@@
 			)
 		)
-		(property "Footprint" "Package_TO_SOT_THT:TO-247-3_Vertical"
+		(property "Footprint" "ac_psu:TO-247-3_Vertical_Proteus"
 			(at 55.88 86.36 0)
 			(effects
@@
 			)
 		)
-		(property "Footprint" "Package_TO_SOT_THT:TO-247-3_Vertical"
+		(property "Footprint" "ac_psu:TO-247-3_Vertical_Proteus"
 			(at 106.68 48.26 0)
 			(effects
@@
 			)
 		)
-		(property "Footprint" "Package_TO_SOT_THT:TO-247-3_Vertical"
+		(property "Footprint" "ac_psu:TO-247-3_Vertical_Proteus"
 			(at 106.68 86.36 0)
 			(effects
@@
 			)
 		)
-		(property "Footprint" "Capacitor_THT:C_Rect_L33.0mm_W20.0mm_P27.50mm_MKS4"
+		(property "Footprint" "ac_psu:C_Rect_L33.0mm_W20.0mm_P27.50mm_MKS4_Proteus"
 			(at 232.1052 59.69 0)
 			(effects
@@
 			)
 		)
-		(property "Footprint" "Capacitor_THT:C_Rect_L33.0mm_W20.0mm_P27.50mm_MKS4"
+		(property "Footprint" "ac_psu:C_Rect_L33.0mm_W20.0mm_P27.50mm_MKS4_Proteus"
 			(at 262.5852 59.69 0)
 			(effects
@@
 			)
 		)
-		(property "Footprint" "Package_SO:TSSOP-8_3x3mm_P0.65mm"
+		(property "Footprint" "ac_psu:TSSOP-8_3x3mm_P0.65mm_Proteus"
 			(at 228.6 106.68 0)
 			(effects
@@
 			)
 		)
-		(property "Footprint" "Package_SO:TSSOP-8_3x3mm_P0.65mm"
+		(property "Footprint" "ac_psu:TSSOP-8_3x3mm_P0.65mm_Proteus"
 			(at 327.66 152.4 0)
 			(effects
@@
 			)
 		)
-		(property "Footprint" "Package_SO:TSSOP-8_3x3mm_P0.65mm"
+		(property "Footprint" "ac_psu:TSSOP-8_3x3mm_P0.65mm_Proteus"
 			(at 38.1 152.4 0)
 			(effects

Commit message: v4 fix 11/12: measurement filters (reports/noise findings 1-5), AMC1306M05
Schematic (sheets 1/3/4/5/9): C95-C106 1n C0G across every 10k leg of the six
difference amplifiers (15.9 kHz tap-node filter), R7 1k -> 10k (U1B + leg
matched; ADA3 scaling changes), R18/R9 100R -> 8.2k with C88/C89 4.7n C0G and
new C107/C108 4.7n on ISOADA1/2 (4.1 kHz), C42/C2 1n -> 10n C0G (1.9 kHz DC
links), C109/C110 100n on REF_1V65/REF_1V65_ISO. R64/DAB series R unchanged
(L unknown; 25R per leg for 10 nH).
Board: fix 11 places the 16 caps (10 top beside their resistor, 6 bottom with
7 vias), renames six auto-named output nets, sets the values; fix 12 re-runs
fix 8's silk placement. DRC 293 (+1 silk), 0 shorts/unconnected/parity.
Deviation rows, v4_copper vias/areas, part map. Replay of fixes 1-12 on the
tag's board gives the board and edit log.
fab: C0G codes C307441/C1518204/C22400107, U4-U6 AMC1306M05DWVR (C701717,
+-50 mV, 4.9k R_IND, checked in SBAS734D), CPL 205 parts, stock for 5 boards
(AMC1306M05: 5 in stock). Noise report: CMTI 50 kV/us min correction.

Co-Authored-By: Claude Opus 5.5 <noreply@anthropic.com>
Claude-Session: https://claude.ai/code/session_01Am5hpeWpvZbzmHWspFiWJm
Parts:
- added C103, C104, C105, C106: 1n C0G, Capacitor_SMD:C_0402_1005Metric, symbol ac_psu:C
- added C107, C108: 4.7n C0G, Capacitor_SMD:C_0402_1005Metric, symbol ac_psu:C
Connections:
- net ISOADA1: now also C107.1
- net ISOADA2: now also C108.1
- net ISOGND: now also C107.2, C108.2
- net REF_1V65_ISO: now also C103.1, C105.1
- net at R52.2, R71.1, U7.3 (+): now also C103.2
- net at R51.2, R68.1, U7.6 (-): now also C106.2
- net at R53.1, R54.2, U7.1: now also C104.1
- net at R256.1, R53.2, U7.2 (-): now also C104.2
- net at R46.2, R67.1, U7.5 (+): now also C105.2
- net at R51.1, R56.2, U7.7: now also C106.1
Other:
- note added: "v4: C103-C106 1n C0G across the 10k legs (15.9 kHz); C107/C108 4.7n on ISOADA1/2 (8.2k/4.7n = 4.1 kHz, v3: none)."
