File: kicad/09_primary_side_adc.kicad_sch (KiCad schematic)
At the start: 0 parts

Commit message: Phase 1: sheet 9 (primary side ADC)
Co-Authored-By: Claude Fable 5.1 <noreply@anthropic.com>
Parts:
- added AD1: ADS7056, symbol ac_psu:ADS7056
- added C17, C18: 100n, symbol ac_psu:C
- added C39: 1u, symbol ac_psu:C
- added C9: 1n, symbol ac_psu:C
- added L1: 22uH, symbol ac_psu:L
- added R86: 10R, symbol ac_psu:R
- added R87: RESISTOR_ARRAY, symbol ac_psu:RESISTOR_ARRAY_4
- added U11: SN74LV4051, symbol ac_psu:SN74LV4051
- added U12: TLV316IDBVR, symbol ac_psu:TLV316IDBVR
Connections:
- new net: AD1.3 (SCLK), R87.6 (R3.2)
- new net: AD1.1 (~{CS}), R87.8 (R1.2)
- new net: AD1.2 (SDO), R87.7 (R2.2)
- new net: R86.2, U12.1, U12.4 (-)
- new net: U11.3 (X), U12.3 (+)
- new net: AD1.4 (DVDD), AD1.6 (AVDD), C17.2, C18.2, L1.1, U12.5 (V+)
- new net: AD1.7 (AINP), C9.2, R86.1
- new net ADA0: U11.15 (X2)
- new net ADA1: U11.14 (X1)
- new net ADA2: U11.13 (X0)
- new net ADA3: U11.12 (X3)
- new net ADA4: U11.1 (X4)
- new net ADA5: U11.2 (X6)
- new net ADA6: U11.4 (X7)
- new net ADASEL0: U11.11 (A)
- new net ADASEL1: U11.10 (B)
- new net ADASEL2: U11.9 (C)
- new net CLK1: R87.3 (R3.1)
- new net CS1: R87.1 (R1.1)
- new net DGND: U11.6 (INH)
- new net GND: AD1.5 (GND), AD1.8 (AINM), C17.1, C18.1, C39.1, C9.1, U11.5 (X5), U11.7 (VEE), U11.8 (VSS), U12.2 (V-)
- new net SDATA1: R87.2 (R2.1)
- new net VCC: C39.2, L1.2, U11.16 (VDD)
- no-connect marks 0 -> 2
Other:
- note added: "AGND and DC- in the Proteus schematic are both net GND; 3V3 = VCC."
- note added: "R87:D (pads 4/5) has no net in the Proteus layout."
- note added: "VDD = 3V3 (VCC), VEE = VSS = AGND (GND); INH tied to the single-pin net DGND."
- note added: "check logic"

Commit message: Phase 2 done: footprints assigned and verified against IPC pads
- tools/gen_footprints.py -> lib/footprint_map.csv + lib/ac_psu.pretty (20 project footprints)
- tools/fpgeom.py: footprint pad loader and rigid fit; tools/check_footprints.py (+ pcbnew
  placement check), added to check_all.sh; reports/footprint_fit.csv for Phase 3 placement
- sch_builder: Footprint field from the map, deterministic UUIDs; all sheets regenerated
- kicad/fp-lib-table; STATUS.md (decisions, residuals, REF3025/C67 findings); Phase 3 prompt

Co-Authored-By: Claude Opus 5.5 <noreply@anthropic.com>
Parts:
- AD1: footprint (none) -> ac_psu:X2QFN-8_1.5x1.5mm_P0.5mm_ADS7056
- C17, C18, C39, C9: footprint (none) -> Capacitor_SMD:C_0402_1005Metric
- L1: footprint (none) -> Inductor_SMD:L_0805_2012Metric
- R86: footprint (none) -> Resistor_SMD:R_0402_1005Metric
- R87: footprint (none) -> ac_psu:R_Array_Convex_4x0402_Proteus
- U11: footprint (none) -> Package_SO:TSSOP-16_4.4x5mm_P0.65mm
- U12: footprint (none) -> ac_psu:SOT-23-5_TLV316
Changed lines of the file:
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@@
 			)
 		)
-		(property "Footprint" ""
+		(property "Footprint" "Capacitor_SMD:C_0402_1005Metric"
 			(at 24.4348 34.29 0)
 			(effects
@@
 			)
 		)
-		(property "Footprint" ""
+		(property "Footprint" "Package_SO:TSSOP-16_4.4x5mm_P0.65mm"
 			(at 63.5 88.9 0)
 			(effects
@@
 			)
 		)
-		(property "Footprint" ""
+		(property "Footprint" "ac_psu:SOT-23-5_TLV316"
 			(at 124.46 78.74 0)
 			(effects
@@
 			)
 		)
-		(property "Footprint" ""
+		(property "Footprint" "Resistor_SMD:R_0402_1005Metric"
 			(at 149.86 71.882 0)
 			(effects
@@
 			)
 		)
-		(property "Footprint" ""
+		(property "Footprint" "Capacitor_SMD:C_0402_1005Metric"
 			(at 159.0548 74.93 0)
 			(effects
@@
 			)
 		)
-		(property "Footprint" ""
+		(property "Footprint" "ac_psu:X2QFN-8_1.5x1.5mm_P0.5mm_ADS7056"
 			(at 215.9 76.2 0)
 			(effects
@@
 			)
 		)
-		(property "Footprint" ""
+		(property "Footprint" "Inductor_SMD:L_0805_2012Metric"
 			(at 190.5 55.88 0)
 			(effects
@@
 			)
 		)
-		(property "Footprint" ""
+		(property "Footprint" "Capacitor_SMD:C_0402_1005Metric"
 			(at 258.1148 64.77 0)
 			(effects
@@
 			)
 		)
-		(property "Footprint" ""
+		(property "Footprint" "Capacitor_SMD:C_0402_1005Metric"
 			(at 265.7348 64.77 0)
 			(effects
@@
 			)
 		)
-		(property "Footprint" ""
+		(property "Footprint" "ac_psu:R_Array_Convex_4x0402_Proteus"
 			(at 236.22 73.152 0)
 			(effects
@@
 			)
 		)
-		(property "Footprint" ""
+		(property "Footprint" "ac_psu:R_Array_Convex_4x0402_Proteus"
 			(at 241.3 88.392 0)
 			(effects
@@
 			)
 		)
-		(property "Footprint" ""
+		(property "Footprint" "ac_psu:R_Array_Convex_4x0402_Proteus"
 			(at 241.3 96.012 0)
 			(effects
@@
 			)
 		)
-		(property "Footprint" ""
+		(property "Footprint" "ac_psu:R_Array_Convex_4x0402_Proteus"
 			(at 241.3 103.632 0)
 			(effects

Commit message: Phase 3 done: PCB rebuilt from the Proteus gerbers with nets and zones
tools/make_pcb.sh regenerates kicad/ac_psu.kicad_pcb (byte-reproducible):
build_pcb.py (footprints with nets and symbol links at the Proteus
positions, outline, mounting holes, rules), gerber_to_tracks.py (4052
tracks, 173 vias; pour edge strokes recognised and skipped),
assign_nets.py (union-find over copper, 0 shorts/orphans/opens with
pours), pours_to_zones.py (79 zones = Proteus pour copper incl. holes).

New checks in check_all.sh: check_board.py (pads/holes/vias vs IPC),
assign_nets.py --check (after zone fill), drc.py (0 shorts, 0
unconnected, 0 parity issues; courtyard overlaps accepted).

Footprints (user decision): Proteus pad sizes for the headers, TSSOP,
SOT-23(-5), SOIC-16W packages whose KiCad pads shorted/violated
clearance; Proteus pads and drills for TO-247, VXO7805, P27.5 film and
snap-in caps; tighter courtyards for IPC-built footprints.

Co-Authored-By: Claude Opus 5.5 <noreply@anthropic.com>
Parts:
- U11: footprint Package_SO:TSSOP-16_4.4x5mm_P0.65mm -> ac_psu:TSSOP-16_4.4x5mm_P0.65mm_Proteus
Changed lines of the file:
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@@
 			)
 		)
-		(property "Footprint" "Package_SO:TSSOP-16_4.4x5mm_P0.65mm"
+		(property "Footprint" "ac_psu:TSSOP-16_4.4x5mm_P0.65mm_Proteus"
 			(at 63.5 88.9 0)
 			(effects

Commit message: v4 design fixes: RET_ISO->ISOGND, U11 INH->GND, C88/C89 on ADA2/ADA3, ADuM7701 RC compensation, R48 Kelvin split
Board frozen: kicad/ac_psu.kicad_pcb edited by one-shot pcbnew scripts tools/v4/fix_1..5
(apply_all.sh, reproducible from the tag's board); make_pcb.sh rebuilds the Proteus board from
tag proteus-conversion-complete into build/proteus/ (byte-identical, checked by regen_check).
Proteus comparisons apply exactly lib/v4_deviations.csv + lib/v4_copper.csv (tools/deviations.py,
wrappers compare_netlists_v4 / check_symbols_v4, deviation support in check_board,
check_footprints, gen_footprints, ipc356_diff, gerber_roundtrip). p2k submodule unchanged.
check_all: ALL CHECKS PASSED; DRC 0 shorts / 0 unconnected / 0 parity (+1 accepted courtyard
overlap C91/U5).

Co-Authored-By: Claude Opus 5.5 <noreply@anthropic.com>
Parts:
- added C88, C89: 1n, Capacitor_SMD:C_0402_1005Metric, symbol ac_psu:C
Connections:
- net DGND is gone; now on net GND: U11.6 (INH)
- net ADA2: now also C88.1
- net ADA3: now also C89.1
- net GND: now also C88.2, C89.2
Other:
- note added: "VDD = 3V3 (VCC), VEE = VSS = AGND (GND)."
- note added: "v4: C88/C89 1n (0402, as C42) filter the mux inputs ADA2/ADA3; placed next to U11."
- note added: "v4: INH (pin 6) tied to GND (v3: single-pin net DGND, floating)."
- note removed: "VDD = 3V3 (VCC), VEE = VSS = AGND (GND); INH tied to the single-pin net DGND."

Commit message: v4 fix 11/12: measurement filters (reports/noise findings 1-5), AMC1306M05
Schematic (sheets 1/3/4/5/9): C95-C106 1n C0G across every 10k leg of the six
difference amplifiers (15.9 kHz tap-node filter), R7 1k -> 10k (U1B + leg
matched; ADA3 scaling changes), R18/R9 100R -> 8.2k with C88/C89 4.7n C0G and
new C107/C108 4.7n on ISOADA1/2 (4.1 kHz), C42/C2 1n -> 10n C0G (1.9 kHz DC
links), C109/C110 100n on REF_1V65/REF_1V65_ISO. R64/DAB series R unchanged
(L unknown; 25R per leg for 10 nH).
Board: fix 11 places the 16 caps (10 top beside their resistor, 6 bottom with
7 vias), renames six auto-named output nets, sets the values; fix 12 re-runs
fix 8's silk placement. DRC 293 (+1 silk), 0 shorts/unconnected/parity.
Deviation rows, v4_copper vias/areas, part map. Replay of fixes 1-12 on the
tag's board gives the board and edit log.
fab: C0G codes C307441/C1518204/C22400107, U4-U6 AMC1306M05DWVR (C701717,
+-50 mV, 4.9k R_IND, checked in SBAS734D), CPL 205 parts, stock for 5 boards
(AMC1306M05: 5 in stock). Noise report: CMTI 50 kV/us min correction.

Co-Authored-By: Claude Opus 5.5 <noreply@anthropic.com>
Claude-Session: https://claude.ai/code/session_01Am5hpeWpvZbzmHWspFiWJm
Parts:
- C88, C89: value 1n -> 4.7n C0G
Other:
- note added: "v4: C88/C89 4.7n C0G (0402) with R18/R9 8.2k filter ADA2/ADA3 at 4.1 kHz; placed next to U11."
- note removed: "v4: C88/C89 1n (0402, as C42) filter the mux inputs ADA2/ADA3; placed next to U11."
Changed lines of the file:
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@@
 			)
 		)
-		(property "Value" "1n"
-			(at 23.96 133.35 0)
+		(property "Value" "4.7n C0G"
+			(at 27.26 133.35 0)
 			(effects
 				(font
@@
 			)
 		)
-		(property "Value" "1n"
-			(at 36.66 133.35 0)
+		(property "Value" "4.7n C0G"
+			(at 39.96 133.35 0)
 			(effects
 				(font
@@
 		)
 	)
-	(text "v4: C88/C89 1n (0402, as C42) filter the mux inputs ADA2/ADA3; placed next to U11."
+	(text "v4: C88/C89 4.7n C0G (0402) with R18/R9 8.2k filter ADA2/ADA3 at 4.1 kHz; placed next to U11."
 		(exclude_from_sim no)
 		(at 12.7 144.78 0)
